Commit message: service bot urdf and gazebo property is edited

File: src/service_description/urdf/servicebot.urdf.xacro (robot description, xacro)
@@ -31,4 +31,25 @@
     <color rgba="0 1 0 1" />
   </material>
+  <material name="yellow">
+    <color rgba="1 1 0 1" />
+  </material>
+  <material name="grey">
+    <color rgba="0.5 0.5 0.5 1" />
+  </material>
+  <material name="orange">
+    <color rgba="1 0.5 0 1" />
+  </material>
+  <material name="brown">
+    <color rgba="0.5 0.25 0 1" />
+  </material>
+  <material name="purple">
+    <color rgba="0.5 0 0.5 1" />
+  </material>
+  <material name="cyan">
+    <color rgba="0 1 1 1" />
+  </material>
+  <material name="magenta">
+    <color rgba="1 0 1 1" />
+  </material>
   <!-- xacro material property -->
   <!-- servicebot -->
@@ -639,5 +660,5 @@
         <geometry>
           <!-- <cylinder length="0.142" radius="0.006" /> -->
-          <mesh filename="package://service_description/meshes/servis/sarhos_tabla.STL" scale="0.001 0.001 0.001" />
+          <mesh filename="package://service_description/meshes/sarhos_tabla/sarhos_tabla.STL" scale="0.001 0.001 0.001" />
         </geometry>
         <origin xyz="-0.03 0.03 -0.035" rpy="1.57079 0 0" />

File: src/service_description/urdf/servicebot_gazebo.urdf.xacro (robot description, xacro)
@@ -47,4 +47,31 @@
 			<maxVel>1.0</maxVel>
 			<material>Gazebo/FlatGray</material>
+		</gazebo>
+		<gazebo reference="base_link">
+			<material>Gazebo/Blue</material>
+		</gazebo>
+		<gazebo reference="upper_chassis">
+			<material>Gazebo/Turquoise</material>
+		</gazebo>
+		<gazebo reference="motor1">
+			<material>Gazebo/Red</material>
+		</gazebo>
+		<gazebo reference="motor2">
+			<material>Gazebo/Red</material>
+		</gazebo>
+		<gazebo reference="motor_baglanti_plaka">
+			<material>Gazebo/Yellow</material>
+		</gazebo>
+		<gazebo reference="motor_baglanti_plaka2">
+			<material>Gazebo/Yellow</material>
+		</gazebo>
+		<gazebo reference="chaster_wheel1">
+			<material>Gazebo/Green</material>
+		</gazebo>
+		<gazebo reference="chaster_wheel2">
+			<material>Gazebo/Green</material>
+		</gazebo>
+		<gazebo reference="chaster_wheel3">
+			<material>Gazebo/Green</material>
 		</gazebo>
 		<!-- This block connects the wheel joint to an actuator (motor), which informs both

Commit message: drive wheells   is edited

File: src/service_description/urdf/servicebot.urdf.xacro (robot description, xacro)
@@ -460,12 +460,12 @@
       <origin xyz="0.04 0.0 0.0" rpy="0 0 0" />
       <parent link="reduktor_mil1" />
-      <child link="reduktor1" />
+      <child link="redüktorteker1" />
       <axis xyz="1 0 0" />
       <!-- <limit lower="-0.15" upper="0.15" effort="100" velocity="0.01" /> -->
     </joint>
-    <link name="reduktor1">
-      <visual>
-        <geometry>
-          <mesh filename="package://service_description/meshes/servis/reduktor.STL" scale="0.001 0.001 0.001" />
+    <link name="redüktorteker">
+      <visual>
+        <geometry>
+          <mesh filename="package://service_description/meshes/servis/reduktorteker.STL" scale="0.001 0.001 0.001" />
         </geometry>
         <origin xyz="-0.155 -0.0725 ${0.0725 + 0.01}" rpy="0 1.57079 0" />
@@ -474,5 +474,5 @@
         <geometry>
           <!-- <cylinder length="0.142" radius="0.006" /> -->
-          <mesh filename="package://service_description/meshes/servis/reduktor.STL" scale="0.001 0.001 0.001" />
+          <mesh filename="package://service_description/meshes/servis/reduktorteker.STL" scale="0.001 0.001 0.001" />
         </geometry>
         <origin xyz="-0.155 -0.0725 ${0.0725 + 0.01}" rpy="0 1.57079 0" />
@@ -496,12 +496,12 @@
       <origin xyz="-0.04 0.0 0.0" rpy="0 0 0" />
       <parent link="reduktor_mil2" />
-      <child link="reduktor2" />
+      <child link="redüktorteker2" />
       <axis xyz="1 0 0" />
       <!-- <limit lower="-0.15" upper="0.15" effort="100" velocity="0.01" /> -->
     </joint>
-    <link name="reduktor2">
-      <visual>
-        <geometry>
-          <mesh filename="package://service_description/meshes/servis/reduktor.STL" scale="0.001 0.001 0.001" />
+    <link name="reduktorteker2">
+      <visual>
+        <geometry>
+          <mesh filename="package://service_description/meshes/servis/reduktorteker.STL" scale="0.001 0.001 0.001" />
         </geometry>
         <origin xyz="0.155 -0.0725 -${0.0725 + 0.01}" rpy="0 -1.57079 0" />
@@ -510,5 +510,5 @@
         <geometry>
           <!-- <cylinder length="0.142" radius="0.006" /> -->
-          <mesh filename="package://service_description/meshes/servis/reduktor.STL" scale="0.001 0.001 0.001" />
+          <mesh filename="package://service_description/meshes/servis/reduktorteker.STL" scale="0.001 0.001 0.001" />
         </geometry>
         <origin xyz="0.155 -0.0725 -${0.0725 + 0.01}" rpy="0 -1.57079 0" />
@@ -528,82 +528,5 @@
       </inertial>
     </link>
-    <!-- Drive Wheel1 -->
-    <joint name="wheel_joint1" type="fixed">
-      <origin xyz="0.0 0.0 0.0" rpy="0 0 0" />
-      <parent link="reduktor1" />
-      <child link="wheel1" />
-      <!-- <axis xyz="0 1 0" /> -->
-      <!-- <limit lower="-0.15" upper="0.15" effort="100" velocity="0.01" /> -->
-    </joint>
-    <link name="wheel1">
-      <visual>
-        <geometry>
-          <mesh filename="package://service_description/meshes/servis/tahrik_tekeri.STL" scale="0.001 0.001 0.001" />
-        </geometry>
-        <origin xyz="-0.155 -0.079 ${0.0725 + 0.01}" rpy="0 1.57079 0" />
-      </visual>
-      <material name="green">
-        <color rgba="0 0 1 1" />
-      </material>
-      <collision>
-        <geometry>
-          <!-- <cylinder length="0.142" radius="0.006" /> -->
-          <mesh filename="package://service_description/meshes/servis/tahrik_tekeri.STL" scale="0.001 0.001 0.001" />
-        </geometry>
-        <origin xyz="-0.155 -0.079 ${0.0725 + 0.01}" rpy="0 1.57079 0" />
-      </collision>
-      <inertial>
-        <!-- COM experimentally determined -->
-        <origin xyz="0.05375 -0.00689  -0.1" />
-        <mass value="0.21" /> <!--  kg for small/big battery pack -->
-        <!-- servicebot's inertia tensor is approximated by a cylinder with homogeneous mass distribution
-             More details: http://en.wikipedia.org/wiki/List_of_moment_of_inertia_tensors
-             m = 2.4 kg; h = 0.09 m; r = 0.175 m
-             ixx = 1/12 * m * (3 * r^2 + h^2)
-             iyy = 1/12 * m * (3 * r^2 + h^2)
-             izz = 1/2 * m * r^2
-          -->
-        <inertia ixx="0.00057724" ixy="0.0" ixz="0.0" iyy="0.00057724" iyz="0.0" izz="0.00000597" />
-      </inertial>
-    </link>
-    <!-- Drive Wheel2 -->
-    <joint name="wheel_joint2" type="fixed">
-      <origin xyz="0.0 0.0 0.0" rpy="0 0 0" />
-      <parent link="reduktor2" />
-      <child link="wheel2" />
-      <!-- <axis xyz="0 1 0" /> -->
-      <!-- <limit lower="-0.15" upper="0.15" effort="100" velocity="0.01" /> -->
-    </joint>
-    <link name="wheel2">
-      <visual>
-        <geometry>
-          <mesh filename="package://service_description/meshes/servis/tahrik_tekeri.STL" scale="0.001 0.001 0.001" />
-        </geometry>
-        <origin xyz="0.155 -0.079 -${0.0725 + 0.01}" rpy="0 -1.57079 0" />
-      </visual>
-      <material name="green">
-        <color rgba="0 0 1 1" />
-      </material>
-      <collision>
-        <geometry>
-          <!-- <cylinder length="0.142" radius="0.006" /> -->
-          <mesh filename="package://service_description/meshes/servis/tahrik_tekeri.STL" scale="0.001 0.001 0.001" />
-        </geometry>
-        <origin xyz="0.155 -0.079 -${0.0725 + 0.01}" rpy="0 -1.57079 0" />
-      </collision>
-      <inertial>
-        <!-- COM experimentally determined -->
-        <origin xyz="0.05375 -0.00689  -0.1" />
-        <mass value="0.21" /> <!--  kg for small/big battery pack -->
-        <!-- servicebot's inertia tensor is approximated by a cylinder with homogeneous mass distribution
-             More details: http://en.wikipedia.org/wiki/List_of_moment_of_inertia_tensors
-             m = 2.4 kg; h = 0.09 m; r = 0.175 m
-             ixx = 1/12 * m * (3 * r^2 + h^2)
-             iyy = 1/12 * m * (3 * r^2 + h^2)
-             izz = 1/2 * m * r^2
-          -->
-        <inertia ixx="0.00057724" ixy="0.0" ixz="0.0" iyy="0.00057724" iyz="0.0" izz="0.00000597" />
-      </inertial>
-    </link>
+    <!-- 3D camera -->
     <!-- Chaster wheel chassis1 -->
     <joint name="chaster_wheel_chassis_joint1" type="revolute">

Commit message: drive wheell2  branch is created for reduktorwheel

File: src/service_description/urdf/servicebot.urdf.xacro (robot description, xacro)
@@ -89,5 +89,5 @@
         <!-- COM experimentally determined -->
         <origin xyz="0.01 0 0" />
-        <mass value="15" /> <!--  kg for small/big battery pack -->
+        <mass value="20" /> <!--  kg for small/big battery pack -->
         <!-- servicebot's inertia tensor is approximated by a cylinder with homogeneous mass distribution
              More details: http://en.wikipedia.org/wiki/List_of_moment_of_inertia_tensors
@@ -236,5 +236,5 @@
       <!-- prismatic -->
       <!-- <origin xyz="0.07 -0.0765 0" rpy="1.5707 0 0 " /> -->
-      <origin xyz="0 -0.0765 -0.04" rpy="0 0 0 " />
+      <origin xyz="0 -0.0765 -0.043" rpy="0 0 0 " />
       <parent link="supan_pole2" />
       <child link="motor_baglanti_plaka" />
@@ -274,5 +274,5 @@
       <!-- prismatic -->
       <!-- <origin xyz="0.07 -0.0765 0" rpy="1.5707 0 0 " /> -->
-      <origin xyz="0 -0.0765 -0.04" rpy="0 0 0 " />
+      <origin xyz="0 -0.0765 -0.043" rpy="0 0 0 " />
       <parent link="supan_pole3" />
       <child link="motor_baglanti_plaka2" />
@@ -348,5 +348,5 @@
     <joint name="motor_joint2" type="fixed">
       <!-- prismatic -->
-      <origin xyz="0.02 0.0 -0.03" rpy="0 0 0" /> <!-- visual and collision, joint shift -->
+      <origin xyz="0.02 0.0 -0.032" rpy="0 0 0" /> <!-- visual and collision, joint shift -->
       <parent link="motor_baglanti_plaka2" />
       <child link="motor2" />
@@ -385,5 +385,5 @@
     <joint name="reduktor_mil_joint1" type="fixed">
       <!-- prismatic -->
-      <origin xyz="0.058 0.0 0.0" rpy="0 0 0" />
+      <origin xyz="0.055 0.0 0.0" rpy="0 0 0" />
       <parent link="motor1" />
       <child link="reduktor_mil1" />
@@ -394,5 +394,5 @@
       <visual>
         <geometry>
-          <mesh filename="package://service_description/meshes/servis/reduktor_mili.STL" scale="0.001 0.001 0.002" />
+          <mesh filename="package://service_description/meshes/servis/reduktor_mili.STL" scale="0.001 0.001 0.001" />
         </geometry>
         <origin xyz="-0.013 -0.007 0.007" rpy="0 1.57079 0" />
@@ -401,5 +401,5 @@
         <geometry>
           <!-- <cylinder length="0.142" radius="0.006" /> -->
-          <mesh filename="package://service_description/meshes/servis/reduktor_mili.STL" scale="0.001 0.001 0.002" />
+          <mesh filename="package://service_description/meshes/servis/reduktor_mili.STL" scale="0.001 0.001 0.001" />
         </geometry>
         <origin xyz="-0.013 -0.007 0.007" rpy="0 1.57079 0" />
@@ -421,5 +421,5 @@
     <!-- Reductor mil2 -->
     <joint name="reduktor_mil_joint2" type="fixed">
-      <origin xyz="-0.058 0.0 0.0" rpy="0 0 0" />
+      <origin xyz="-0.055 0.0 0.0" rpy="0 0 0" />
       <parent link="motor2" />
       <child link="reduktor_mil2" />
@@ -430,5 +430,5 @@
       <visual>
         <geometry>
-          <mesh filename="package://service_description/meshes/servis/reduktor_mili.STL" scale="0.001 0.001 0.002" />
+          <mesh filename="package://service_description/meshes/servis/reduktor_mili.STL" scale="0.001 0.001 0.001" />
         </geometry>
         <origin xyz="0.013 -0.007 -0.007" rpy="0 -1.57079 0" />
@@ -437,5 +437,5 @@
         <geometry>
           <!-- <cylinder length="0.142" radius="0.006" /> -->
-          <mesh filename="package://service_description/meshes/servis/reduktor_mili.STL" scale="0.001 0.001 0.002" />
+          <mesh filename="package://service_description/meshes/servis/reduktor_mili.STL" scale="0.001 0.001 0.001" />
         </geometry>
         <origin xyz="0.013 -0.007 -0.007" rpy="0 -1.57079 0" />
@@ -460,14 +460,15 @@
       <origin xyz="0.04 0.0 0.0" rpy="0 0 0" />
       <parent link="reduktor_mil1" />
-      <child link="redüktorteker1" />
+      <child link="reduktorteker1" />
       <axis xyz="1 0 0" />
       <!-- <limit lower="-0.15" upper="0.15" effort="100" velocity="0.01" /> -->
-    </joint>
-    <link name="redüktorteker">
+      <limit effort="100" velocity="20" />
+    </joint>
+    <link name="reduktorteker1">
       <visual>
         <geometry>
           <mesh filename="package://service_description/meshes/servis/reduktorteker.STL" scale="0.001 0.001 0.001" />
         </geometry>
-        <origin xyz="-0.155 -0.0725 ${0.0725 + 0.01}" rpy="0 1.57079 0" />
+        <origin xyz="-0.155 -0.079 ${0.0725 + 0.01}" rpy="0 1.57079 0" />
       </visual>
       <collision>
@@ -476,5 +477,5 @@
           <mesh filename="package://service_description/meshes/servis/reduktorteker.STL" scale="0.001 0.001 0.001" />
         </geometry>
-        <origin xyz="-0.155 -0.0725 ${0.0725 + 0.01}" rpy="0 1.57079 0" />
+        <origin xyz="-0.155 -0.079 ${0.0725 + 0.01}" rpy="0 1.57079 0" />
       </collision>
       <inertial>
@@ -496,7 +497,8 @@
       <origin xyz="-0.04 0.0 0.0" rpy="0 0 0" />
       <parent link="reduktor_mil2" />
-      <child link="redüktorteker2" />
+      <child link="reduktorteker2" />
       <axis xyz="1 0 0" />
       <!-- <limit lower="-0.15" upper="0.15" effort="100" velocity="0.01" /> -->
+      <limit effort="100" velocity="20" />
     </joint>
     <link name="reduktorteker2">
@@ -505,5 +507,5 @@
           <mesh filename="package://service_description/meshes/servis/reduktorteker.STL" scale="0.001 0.001 0.001" />
         </geometry>
-        <origin xyz="0.155 -0.0725 -${0.0725 + 0.01}" rpy="0 -1.57079 0" />
+        <origin xyz="0.155 -0.079 -${0.0725 + 0.01}" rpy="0 -1.57079 0" />
       </visual>
       <collision>
@@ -512,5 +514,5 @@
           <mesh filename="package://service_description/meshes/servis/reduktorteker.STL" scale="0.001 0.001 0.001" />
         </geometry>
-        <origin xyz="0.155 -0.0725 -${0.0725 + 0.01}" rpy="0 -1.57079 0" />
+        <origin xyz="0.155 -0.079 -${0.0725 + 0.01}" rpy="0 -1.57079 0" />
       </collision>
       <inertial>
@@ -535,5 +537,6 @@
       <child link="chaster_wheel_chassis1" />
       <axis xyz="0 0 1" />
-      <limit lower="-3.1415926" upper="3.1415926" effort="100" velocity="0.1" />
+      <limit lower="3.14159" upper="3.14159" effort="10" velocity="1" />
+      <dynamics damping="0.01" friction="0.0" />
     </joint>
     <link name="chaster_wheel_chassis1">
@@ -571,5 +574,6 @@
       <child link="chaster_wheel_chassis2" />
       <axis xyz="0 0 1" />
-      <limit lower="-3.1415926" upper="3.1415926" effort="100" velocity="0.1" />
+      <limit lower="-3.14" upper="3.14" effort="10" velocity="1" />
+      <dynamics damping="0.01" friction="0.0" />
     </joint>
     <link name="chaster_wheel_chassis2">
@@ -607,5 +611,6 @@
       <child link="chaster_wheel_chassis3" />
       <axis xyz="0 0 1" />
-      <limit lower="-3.1415926" upper="3.1415926" effort="100" velocity="0.1" />
+      <limit lower="-3.14" upper="3.14" effort="10" velocity="1" />
+      <dynamics damping="0.01" friction="0.0" />
     </joint>
     <link name="chaster_wheel_chassis3">
@@ -643,4 +648,5 @@
       <child link="chaster_wheel1" />
       <axis xyz="1 0 0" />
+      <limit lower="-3.14" upper="3.14" effort="100" velocity="20" />
       <dynamics damping="0.1" friction="0.1" />
     </joint>
@@ -780,13 +786,13 @@
         <!-- COM experimentally determined -->
         <origin xyz="0.0 0.0 0.0" />
-        <mass value="0.20" /> <!--  kg for small/big battery pack -->
-        <!-- servicebot's inertia tensor is approximated by a cylinder with homogeneous mass distribution
-             More details: http://en.wikipedia.org/wiki/List_of_moment_of_inertia_tensors
-             m = 2.4 kg; h = 0.09 m; r = 0.175 m
-             ixx = 1/12 * m * (3 * r^2 + h^2)
-             iyy = 1/12 * m * (3 * r^2 + h^2)
-             izz = 1/2 * m * r^2
-          -->
-        <inertia ixx="0.00057724" ixy="0.0" ixz="0.0" iyy="0.00057724" iyz="0.0" izz="0.00000597" />
+        <mass value="30" /> <!--  kg for small/big battery pack -->
+        <!-- servicebot's inertia tensor is approximated by a cylinder with homogeneous mass distribution
+             More details: http://en.wikipedia.org/wiki/List_of_moment_of_inertia_tensors
+             m = 2.4 kg; h = 0.09 m; r = 0.175 m
+             ixx = 1/12 * m * (3 * r^2 + h^2)
+             iyy = 1/12 * m * (3 * r^2 + h^2)
+             izz = 1/2 * m * r^2
+          -->
+        <inertia ixx="0.0057724" ixy="0.0" ixz="0.0" iyy="0.0057724" iyz="0.0" izz="0.0000597" />
       </inertial>
     </link>

File: src/service_description/urdf/servicebot_gazebo.urdf.xacro (robot description, xacro)
@@ -2,52 +2,57 @@
 <robot name="servicebot_sim" xmlns:xacro="http://www.ros.org/wiki/xacro">
 	<xacro:macro name="servicebot_sim">
-		<gazebo reference="reduktor1">
-			<mu1>1.0</mu1>
-			<mu2>1.0</mu2>
-			<kp>1000000.0</kp>
-			<kd>100.0</kd>
+		<gazebo reference="base_link">
+			<material>Gazebo/Blue</material>
+		</gazebo>
+		<gazebo reference="reduktorteker1">
+			<mu1 value="200.0" />
+			<mu2 value="100.0" />
+			<kp value="10000000.0" />
+			<kd value="1.0" />
 			<minDepth>0.001</minDepth>
 			<maxVel>1.0</maxVel>
 			<maxForce>1000.0</maxForce>
-			<material>Gazebo/Blue</material>
+			<material>Gazebo/Green</material>
+			<turnGravityOff>false</turnGravityOff>
 		</gazebo>
-		<gazebo reference="reduktor2">
-			<mu1>1.0</mu1>
-			<mu2>1.0</mu2>
-			<kp>1000000.0</kp>
-			<kd>100.0</kd>
+		<gazebo reference="reduktorteker2">
+			<mu1 value="200.0" />
+			<mu2 value="100.0" />
+			<kp value="10000000.0" />
+			<kd value="1.0" />
 			<minDepth>0.001</minDepth>
 			<maxVel>1.0</maxVel>
-			<material>Gazebo/Blue</material>
+			<material>Gazebo/Green</material>
+			<turnGravityOff>false</turnGravityOff>
 		</gazebo>
 		<gazebo reference="chaster_wheel1">
-			<mu1>0.0</mu1>
-			<mu2>0.0</mu2>
-			<kp>1000000.0</kp>
-			<kd>100.0</kd>
+			<mu1 value="200.0" />
+			<mu2 value="100.0" />
+			<kp value="10000000.0" />
+			<kd value="1.0" />
 			<minDepth>0.001</minDepth>
 			<maxVel>1.0</maxVel>
-			<material>Gazebo/FlatGray</material>
+			<material>Gazebo/Green</material>
+			<turnGravityOff>false</turnGravityOff>
 		</gazebo>
 		<gazebo reference="chaster_wheel2">
-			<mu1>0.0</mu1>
-			<mu2>0.0</mu2>
-			<kp>1000000.0</kp>
-			<kd>100.0</kd>
+			<mu1 value="200.0" />
+			<mu2 value="100.0" />
+			<kp value="10000000.0" />
+			<kd value="1.0" />
 			<minDepth>0.001</minDepth>
 			<maxVel>1.0</maxVel>
-			<material>Gazebo/FlatGray</material>
+			<material>Gazebo/Green</material>
+			<turnGravityOff>false</turnGravityOff>
 		</gazebo>
 		<gazebo reference="chaster_wheel3">
-			<mu1>0.0</mu1>
-			<mu2>0.0</mu2>
-			<kp>1000000.0</kp>
-			<kd>100.0</kd>
+			<mu1 value="200.0" />
+			<mu2 value="100.0" />
+			<kp value="10000000.0" />
+			<kd value="1.0" />
 			<minDepth>0.001</minDepth>
 			<maxVel>1.0</maxVel>
-			<material>Gazebo/FlatGray</material>
-		</gazebo>
-		<gazebo reference="base_link">
-			<material>Gazebo/Blue</material>
+			<material>Gazebo/Green</material>
+			<turnGravityOff>false</turnGravityOff>
 		</gazebo>
 		<gazebo reference="upper_chassis">
@@ -66,13 +71,4 @@
 			<material>Gazebo/Yellow</material>
 		</gazebo>
-		<gazebo reference="chaster_wheel1">
-			<material>Gazebo/Green</material>
-		</gazebo>
-		<gazebo reference="chaster_wheel2">
-			<material>Gazebo/Green</material>
-		</gazebo>
-		<gazebo reference="chaster_wheel3">
-			<material>Gazebo/Green</material>
-		</gazebo>
 		<!-- This block connects the wheel joint to an actuator (motor), which informs both
     simulation and visualization of the robot -->
@@ -80,8 +76,8 @@
 			<type>transmission_interface/SimpleTransmission</type>
 			<actuator name="wheel_motor2">
-				<mechanicalReduction>21</mechanicalReduction>
+				<mechanicalReduction>1</mechanicalReduction>
 			</actuator>
-			<joint name="$reduktor_joint2">
-				<hardwareInterface>VelocityJointInterface</hardwareInterface>
+			<joint name="reduktor_joint2">
+				<hardwareInterface>hardware_interface/VelocityJointInterface</hardwareInterface>
 			</joint>
 		</transmission>
@@ -89,31 +85,39 @@
 			<type>transmission_interface/SimpleTransmission</type>
 			<actuator name="wheel_motor1">
-				<mechanicalReduction>21</mechanicalReduction>
+				<mechanicalReduction>1</mechanicalReduction>
 			</actuator>
 			<joint name="reduktor_joint1">
-				<hardwareInterface>VelocityJointInterface</hardwareInterface>
+				<hardwareInterface>hardware_interface/VelocityJointInterface</hardwareInterface>
 			</joint>
 		</transmission>
 		<!-- Gazebo plugin for ROS Control -->
-		<gazebo>
+		<!-- <gazebo>
 			<plugin name="gazebo_ros_control" filename="libgazebo_ros_control.so">
 				<robotNamespace>/</robotNamespace>
 			</plugin>
-		</gazebo>
+		</gazebo> -->
 		<gazebo>
-			<plugin name="differential_drive_controller" filename="libgazebo_ros_diff_drive.so">
+			<plugin filename="libgazebo_ros_diff_drive.so" name="differential_drive_controller">
 				<alwaysOn>true</alwaysOn>
 				<updateRate>20</updateRate>
-				<leftJoint>reduktor_joint2</leftJoint>
+				<publishTf> true </publishTf>
+				<leftJoint>reduktor_joint1</leftJoint>
 				<rightJoint>reduktor_joint2</rightJoint>
 				<wheelSeparation>.230</wheelSeparation>
 				<wheelDiameter>0.070</wheelDiameter>
-				<torque>1.0</torque>
-				<commandTopic>cmd_vel</commandTopic>
-				<odometryTopic>odom</odometryTopic>
-				<odometryFrame>odom</odometryFrame>
-				<robotBaseFrame>base_footprint</robotBaseFrame>
+				<torque>5.0</torque>
+				<commandTopic>/cmd_vel</commandTopic>
+				<odometrySource>world</odometrySource> <!-- 'encoder' instead of 'world' is also possible -->
+				<odometryTopic>/odom</odometryTopic> <!-- relative/name ,  /global/name  -->
+				<odometryFrame>/odom</odometryFrame>
+				<robotBaseFrame>/base_footprint</robotBaseFrame>
+				<publishOdomTF> true </publishOdomTF>
 				<publishWheelJointState>true</publishWheelJointState>
+				<!-- Set to true to publish transforms for the wheel links, defaults to false -->
+				<publishWheelTF>false</publishWheelTF>
+				<wheelAcceleration> 2.8 </wheelAcceleration>
+				<wheelTorque> 5.0 </wheelTorque>
 				<legacyMode>true</legacyMode>
+				<rosDebugLevel> Debug </rosDebugLevel> <!-- <rosDebugLevel>Debug</rosDebugLevel> -->
 			</plugin>
 		</gazebo>
