Commit message: add gazebo diff drive configurations

File: src/service_description/urdf/servicebot.urdf.xacro (robot description, xacro)
@@ -1,8 +1,8 @@
 <?xml version="1.0"?>
 <!--
-  This is not a standalone urdf for servicebot. It simply defines the 'servicebot' tag that can
+  This is not a standalone urdf for kobuki. It simply defines the 'kobuki' tag that can
   be incorporated by other urdf files (e.g. turtlebot).
-  See servicebot_standalone.urdf.xacro for a standalone urdf to be tested with
-      servicebot_description/launch/view_model.launch
+  See kobuki_standalone.urdf.xacro for a standalone urdf to be tested with
+      kobuki_description/launch/view_model.launch
  -->
 <robot name="servicebot" xmlns:xacro="http://www.ros.org/wiki/xacro">
@@ -26,11 +26,11 @@
   </material>
   <material name="red">
-    <color rgba="1 0 0 1" />
+    <color rgba="0.8 0 0 1" />
   </material>
   <material name="green">
-    <color rgba="0 1 0 1" />
+    <color rgba="0 0.8 0 1" />
   </material>
   <material name="yellow">
-    <color rgba="1 1 0 1" />
+    <color rgba="0.8 0.8 0 1" />
   </material>
   <material name="grey">
@@ -38,20 +38,35 @@
   </material>
   <material name="orange">
-    <color rgba="1 0.5 0 1" />
+    <color rgba="0.8 0.5 0 1" />
   </material>
   <material name="brown">
     <color rgba="0.5 0.25 0 1" />
   </material>
+  <material name="silver">
+    <color rgba="0.75 0.75 0.75 1" />
+  </material>
+  <material name="gold">
+    <color rgba="0.75 0.75 0 1" />
+  </material>
+  <material name="cyan">
+    <color rgba="0 0.8 0.8 1" />
+  </material>
+  <material name="magenta">
+    <color rgba="0.8 0 0.8 1" />
+  </material>
   <material name="purple">
     <color rgba="0.5 0 0.5 1" />
   </material>
-  <material name="cyan">
-    <color rgba="0 1 1 1" />
-  </material>
-  <material name="magenta">
-    <color rgba="1 0 1 1" />
+  <material name="pink">
+    <color rgba="0.8 0.5 0.5 1" />
+  </material>
+  <material name="lightblue">
+    <color rgba="0.5 0.5 0.8 1" />
+  </material>
+  <material name="bronze">
+    <color rgba="0.8 0.5 0.25 1" />
   </material>
   <!-- xacro material property -->
-  <!-- servicebot -->
+  <!-- Kobuki -->
   <xacro:macro name="servicebot">
     <link name="base_footprint" />
@@ -76,5 +91,5 @@
           <mesh filename="package://service_description/meshes/servis/sase2.STL" scale="0.001 0.001 0.001" />
         </geometry>
-        <material name="blue" />
+        <material name="silver" />
         <origin xyz="-0.237 -0.254  -0.281" rpy="0 0 0" />
       </visual>
@@ -90,5 +105,5 @@
         <origin xyz="0.01 0 0" />
         <mass value="15" /> <!--  kg for small/big battery pack -->
-        <!-- servicebot's inertia tensor is approximated by a cylinder with homogeneous mass distribution
+        <!-- Kobuki's inertia tensor is approximated by a cylinder with homogeneous mass distribution
              More details: http://en.wikipedia.org/wiki/List_of_moment_of_inertia_tensors
              m = 2.4 kg; h = 0.09 m; r = 0.175 m
@@ -111,4 +126,5 @@
         </geometry>
         <origin xyz="-0.006 -0.006 -0.071" rpy="0 0 0" />
+        <material name="purple" />
       </visual>
       <collision>
@@ -123,5 +139,5 @@
         <origin xyz="0.1455 0.0765 0.141" />
         <mass value="0.21" /> <!--  kg for small/big battery pack -->
-        <!-- servicebot's inertia tensor is approximated by a cylinder with homogeneous mass distribution
+        <!-- Kobuki's inertia tensor is approximated by a cylinder with homogeneous mass distribution
              More details: http://en.wikipedia.org/wiki/List_of_moment_of_inertia_tensors
              m = 2.4 kg; h = 0.09 m; r = 0.175 m
@@ -144,4 +160,5 @@
         </geometry>
         <origin xyz="-0.006 -0.006 -0.071" rpy="0 0 0" />
+        <material name="purple" />
       </visual>
       <collision>
@@ -156,5 +173,5 @@
         <origin xyz="-0.1455 -0.0765  0.141" />
         <mass value="0.21" /> <!--  kg for small/big battery pack -->
-        <!-- servicebot's inertia tensor is approximated by a cylinder with homogeneous mass distribution
+        <!-- Kobuki's inertia tensor is approximated by a cylinder with homogeneous mass distribution
              More details: http://en.wikipedia.org/wiki/List_of_moment_of_inertia_tensors
              m = 2.4 kg; h = 0.09 m; r = 0.175 m
@@ -177,4 +194,5 @@
         </geometry>
         <origin xyz="-0.006 -0.006 -0.071" rpy="0 0 0" />
+        <material name="purple" />
       </visual>
       <collision>
@@ -189,5 +207,5 @@
         <origin xyz="-0.1455 0.0765 0.141" />
         <mass value="0.21" /> <!--  kg for small/big battery pack -->
-        <!-- servicebot's inertia tensor is approximated by a cylinder with homogeneous mass distribution
+        <!-- Kobuki's inertia tensor is approximated by a cylinder with homogeneous mass distribution
              More details: http://en.wikipedia.org/wiki/List_of_moment_of_inertia_tensors
              m = 2.4 kg; h = 0.09 m; r = 0.175 m
@@ -210,4 +228,5 @@
         </geometry>
         <origin xyz="-0.006 -0.006 -0.071" rpy="0 0 0" />
+        <material name="purple" />
       </visual>
       <collision>
@@ -222,5 +241,5 @@
         <origin xyz="0.1455 -0.0765 0.141" />
         <mass value="0.21" /> <!--  kg for small/big battery pack -->
-        <!-- servicebot's inertia tensor is approximated by a cylinder with homogeneous mass distribution
+        <!-- Kobuki's inertia tensor is approximated by a cylinder with homogeneous mass distribution
              More details: http://en.wikipedia.org/wiki/List_of_moment_of_inertia_tensors
              m = 2.4 kg; h = 0.09 m; r = 0.175 m
@@ -248,4 +267,5 @@
         </geometry>
         <origin xyz="-0.015  0.176 -0.086" rpy="1.5707 0 0" />
+        <material name="gold" />
       </visual>
       <collision>
@@ -260,5 +280,5 @@
         <origin xyz="0.05375 -0.00689  -0.1" />
         <mass value="0.21" /> <!--  kg for small/big battery pack -->
-        <!-- servicebot's inertia tensor is approximated by a cylinder with homogeneous mass distribution
+        <!-- Kobuki's inertia tensor is approximated by a cylinder with homogeneous mass distribution
              More details: http://en.wikipedia.org/wiki/List_of_moment_of_inertia_tensors
              m = 2.4 kg; h = 0.09 m; r = 0.175 m
@@ -286,4 +306,5 @@
         </geometry>
         <origin xyz="0.015  -0.176 -0.086" rpy="1.5707 0 -3.1415926" />
+        <material name="gold" />
       </visual>
       <collision>
@@ -298,5 +319,5 @@
         <origin xyz="0.05375 -0.00689  -0.1" />
         <mass value="0.21" /> <!--  kg for small/big battery pack -->
-        <!-- servicebot's inertia tensor is approximated by a cylinder with homogeneous mass distribution
+        <!-- Kobuki's inertia tensor is approximated by a cylinder with homogeneous mass distribution
              More details: http://en.wikipedia.org/wiki/List_of_moment_of_inertia_tensors
              m = 2.4 kg; h = 0.09 m; r = 0.175 m
@@ -323,4 +344,5 @@
         </geometry>
         <origin xyz="-0.04 -0.03 0.03" rpy="0 1.57079 0" />
+        <material name="black" />
       </visual>
       <collision>
@@ -335,5 +357,5 @@
         <origin xyz="0.05375 -0.00689  -0.1" />
         <mass value="0.21" /> <!--  kg for small/big battery pack -->
-        <!-- servicebot's inertia tensor is approximated by a cylinder with homogeneous mass distribution
+        <!-- Kobuki's inertia tensor is approximated by a cylinder with homogeneous mass distribution
              More details: http://en.wikipedia.org/wiki/List_of_moment_of_inertia_tensors
              m = 2.4 kg; h = 0.09 m; r = 0.175 m
@@ -360,4 +382,5 @@
         </geometry>
         <origin xyz="0.04 -0.03 -0.03" rpy="0 -1.57079 0" />
+        <material name="black" />
       </visual>
       <collision>
@@ -372,5 +395,5 @@
         <origin xyz="0.05375 -0.00689  -0.1" />
         <mass value="0.21" /> <!--  kg for small/big battery pack -->
-        <!-- servicebot's inertia tensor is approximated by a cylinder with homogeneous mass distribution
+        <!-- Kobuki's inertia tensor is approximated by a cylinder with homogeneous mass distribution
              More details: http://en.wikipedia.org/wiki/List_of_moment_of_inertia_tensors
              m = 2.4 kg; h = 0.09 m; r = 0.175 m
@@ -397,4 +420,5 @@
         </geometry>
         <origin xyz="-0.013 -0.007 0.007" rpy="0 1.57079 0" />
+        <material name="magenta" />
       </visual>
       <collision>
@@ -409,5 +433,5 @@
         <origin xyz="0.05375 -0.00689  -0.1" />
         <mass value="0.21" /> <!--  kg for small/big battery pack -->
-        <!-- servicebot's inertia tensor is approximated by a cylinder with homogeneous mass distribution
+        <!-- Kobuki's inertia tensor is approximated by a cylinder with homogeneous mass distribution
              More details: http://en.wikipedia.org/wiki/List_of_moment_of_inertia_tensors
              m = 2.4 kg; h = 0.09 m; r = 0.175 m
@@ -433,4 +457,5 @@
         </geometry>
         <origin xyz="0.013 -0.007 -0.007" rpy="0 -1.57079 0" />
+        <material name="magenta" />
       </visual>
       <collision>
@@ -445,5 +470,5 @@
         <origin xyz="0.05375 -0.00689  -0.1" />
         <mass value="0.21" /> <!--  kg for small/big battery pack -->
-        <!-- servicebot's inertia tensor is approximated by a cylinder with homogeneous mass distribution
+        <!-- Kobuki's inertia tensor is approximated by a cylinder with homogeneous mass distribution
              More details: http://en.wikipedia.org/wiki/List_of_moment_of_inertia_tensors
              m = 2.4 kg; h = 0.09 m; r = 0.175 m
@@ -458,6 +483,6 @@
     <joint name="reduktor_joint1" type="continuous">
       <!-- prismatic -->
-      <origin xyz="0.04 0.0 0.0" rpy="0 0 0" />
-      <parent link="reduktor_mil1" />
+      <origin xyz="0.24 0.0 0.0777" rpy="0 0 0" />
+      <parent link="base_link" />
       <child link="reduktor1" />
       <axis xyz="1 0 0" />
@@ -469,5 +494,6 @@
           <mesh filename="package://service_description/meshes/servis/reduktor.STL" scale="0.001 0.001 0.001" />
         </geometry>
-        <origin xyz="-0.155 -0.0725 ${0.0725 + 0.01}" rpy="0 1.57079 0" />
+        <origin xyz="-0.155 -0.073 ${0.0725 + 0.01}" rpy="0 1.57079 0" />
+        <material name="cyan" />
       </visual>
       <collision>
@@ -476,11 +502,11 @@
           <mesh filename="package://service_description/meshes/servis/reduktor.STL" scale="0.001 0.001 0.001" />
         </geometry>
-        <origin xyz="-0.155 -0.0725 ${0.0725 + 0.01}" rpy="0 1.57079 0" />
-      </collision>
-      <inertial>
-        <!-- COM experimentally determined -->
-        <origin xyz="0.05375 -0.00689  -0.1" />
-        <mass value="0.21" /> <!--  kg for small/big battery pack -->
-        <!-- servicebot's inertia tensor is approximated by a cylinder with homogeneous mass distribution
+        <origin xyz="-0.155 -0.073 ${0.0725 + 0.01}" rpy="0 1.57079 0" />
+      </collision>
+      <inertial>
+        <!-- COM experimentally determined -->
+        <origin xyz="0.05375 -0.00689  -0.1" />
+        <mass value="0.21" /> <!--  kg for small/big battery pack -->
+        <!-- Kobuki's inertia tensor is approximated by a cylinder with homogeneous mass distribution
              More details: http://en.wikipedia.org/wiki/List_of_moment_of_inertia_tensors
              m = 2.4 kg; h = 0.09 m; r = 0.175 m
@@ -494,6 +520,6 @@
     <!-- reduktor2 -->
     <joint name="reduktor_joint2" type="continuous">
-      <origin xyz="-0.04 0.0 0.0" rpy="0 0 0" />
-      <parent link="reduktor_mil2" />
+      <origin xyz="-0.24 0.0 0.0777" rpy="0 0 0" />
+      <parent link="base_link" />
       <child link="reduktor2" />
       <axis xyz="1 0 0" />
@@ -505,5 +531,6 @@
           <mesh filename="package://service_description/meshes/servis/reduktor.STL" scale="0.001 0.001 0.001" />
         </geometry>
-        <origin xyz="0.155 -0.0725 -${0.0725 + 0.01}" rpy="0 -1.57079 0" />
+        <origin xyz="0.155 -0.073 -${0.0725 + 0.01}" rpy="0 -1.57079 0" />
+        <material name="cyan" />
       </visual>
       <collision>
@@ -512,11 +539,11 @@
           <mesh filename="package://service_description/meshes/servis/reduktor.STL" scale="0.001 0.001 0.001" />
         </geometry>
-        <origin xyz="0.155 -0.0725 -${0.0725 + 0.01}" rpy="0 -1.57079 0" />
-      </collision>
-      <inertial>
-        <!-- COM experimentally determined -->
-        <origin xyz="0.05375 -0.00689  -0.1" />
-        <mass value="0.21" /> <!--  kg for small/big battery pack -->
-        <!-- servicebot's inertia tensor is approximated by a cylinder with homogeneous mass distribution
+        <origin xyz="0.155 -0.073 -${0.0725 + 0.01}" rpy="0 -1.57079 0" />
+      </collision>
+      <inertial>
+        <!-- COM experimentally determined -->
+        <origin xyz="0.05375 -0.00689  -0.1" />
+        <mass value="0.21" /> <!--  kg for small/big battery pack -->
+        <!-- Kobuki's inertia tensor is approximated by a cylinder with homogeneous mass distribution
              More details: http://en.wikipedia.org/wiki/List_of_moment_of_inertia_tensors
              m = 2.4 kg; h = 0.09 m; r = 0.175 m
@@ -542,8 +569,6 @@
         </geometry>
         <origin xyz="-0.155 -0.079 ${0.0725 + 0.01}" rpy="0 1.57079 0" />
-      </visual>
-      <material name="green">
-        <color rgba="0 0 1 1" />
-      </material>
+        <material name="green" />
+      </visual>
       <collision>
         <geometry>
@@ -551,11 +576,11 @@
           <mesh filename="package://service_description/meshes/servis/tahrik_tekeri.STL" scale="0.001 0.001 0.001" />
         </geometry>
-        <origin xyz="-0.155 -0.079 ${0.0725 + 0.01}" rpy="0 1.57079 0" />
-      </collision>
-      <inertial>
-        <!-- COM experimentally determined -->
-        <origin xyz="0.05375 -0.00689  -0.1" />
-        <mass value="0.21" /> <!--  kg for small/big battery pack -->
-        <!-- servicebot's inertia tensor is approximated by a cylinder with homogeneous mass distribution
+        <origin xyz="-0.155 -0.07 ${0.0725 + 0.01}" rpy="0 1.57079 0" />
+      </collision>
+      <inertial>
+        <!-- COM experimentally determined -->
+        <origin xyz="0.05375 -0.00689  -0.1" />
+        <mass value="0.21" /> <!--  kg for small/big battery pack -->
+        <!-- Kobuki's inertia tensor is approximated by a cylinder with homogeneous mass distribution
              More details: http://en.wikipedia.org/wiki/List_of_moment_of_inertia_tensors
              m = 2.4 kg; h = 0.09 m; r = 0.175 m
@@ -581,8 +606,6 @@
         </geometry>
         <origin xyz="0.155 -0.079 -${0.0725 + 0.01}" rpy="0 -1.57079 0" />
-      </visual>
-      <material name="green">
-        <color rgba="0 0 1 1" />
-      </material>
+        <material name="green" />
+      </visual>
       <collision>
         <geometry>
@@ -596,5 +619,5 @@
         <origin xyz="0.05375 -0.00689  -0.1" />
         <mass value="0.21" /> <!--  kg for small/big battery pack -->
-        <!-- servicebot's inertia tensor is approximated by a cylinder with homogeneous mass distribution
+        <!-- Kobuki's inertia tensor is approximated by a cylinder with homogeneous mass distribution
              More details: http://en.wikipedia.org/wiki/List_of_moment_of_inertia_tensors
              m = 2.4 kg; h = 0.09 m; r = 0.175 m
@@ -607,10 +630,10 @@
     </link>
     <!-- Chaster wheel chassis1 -->
-    <joint name="chaster_wheel_chassis_joint1" type="revolute">
+    <joint name="chaster_wheel_chassis_joint1" type="continuous">
       <origin xyz="0.006 -0.198 0.047" rpy="0 0 0 " />
       <parent link="base_link" />
       <child link="chaster_wheel_chassis1" />
       <axis xyz="0 0 1" />
-      <limit lower="-3.1415926" upper="3.1415926" effort="100" velocity="0.1" />
+      <dynamics damping="0.01" friction="0.0" />
     </joint>
     <link name="chaster_wheel_chassis1">
@@ -620,4 +643,5 @@
         </geometry>
         <origin xyz="-0.03 0.03 -0.035" rpy="1.57079 0 0" />
+        <material name="brown" />
       </visual>
       <collision>
@@ -632,5 +656,5 @@
         <origin xyz="0.0 0.0 0.0" />
         <mass value="0.21" /> <!--  kg for small/big battery pack -->
-        <!-- servicebot's inertia tensor is approximated by a cylinder with homogeneous mass distribution
+        <!-- Kobuki's inertia tensor is approximated by a cylinder with homogeneous mass distribution
              More details: http://en.wikipedia.org/wiki/List_of_moment_of_inertia_tensors
              m = 2.4 kg; h = 0.09 m; r = 0.175 m
@@ -643,10 +667,10 @@
     </link>
     <!-- Chaster wheel chassis2 -->
-    <joint name="chaster_wheel_chassis_joint2" type="revolute">
+    <joint name="chaster_wheel_chassis_joint2" type="continuous">
       <origin xyz="-0.115 0.156 0.047" rpy="0 0 0 " />
       <parent link="base_link" />
       <child link="chaster_wheel_chassis2" />
       <axis xyz="0 0 1" />
-      <limit lower="-3.1415926" upper="3.1415926" effort="100" velocity="0.1" />
+      <dynamics damping="0.01" friction="0.0" />
     </joint>
     <link name="chaster_wheel_chassis2">
@@ -656,9 +680,10 @@
         </geometry>
         <origin xyz="-0.03 0.03 -0.035" rpy="1.57079 0 0" />
-      </visual>
-      <collision>
-        <geometry>
-          <!-- <cylinder length="0.142" radius="0.006" /> -->
-          <mesh filename="package://service_description/meshes/sarhos_tabla/sarhos_tabla.STL" scale="0.001 0.001 0.001" />
+        <material name="brown" />
+      </visual>
+      <collision>
+        <geometry>
+          <!-- <cylinder length="0.142" radius="0.006" /> -->
+          <mesh filename="package://service_description/meshes/servis/sarhos_tabla.STL" scale="0.001 0.001 0.001" />
         </geometry>
         <origin xyz="-0.03 0.03 -0.035" rpy="1.57079 0 0" />
@@ -668,5 +693,5 @@
         <origin xyz="0.0 0.0 0.0" />
         <mass value="0.21" /> <!--  kg for small/big battery pack -->
-        <!-- servicebot's inertia tensor is approximated by a cylinder with homogeneous mass distribution
+        <!-- Kobuki's inertia tensor is approximated by a cylinder with homogeneous mass distribution
              More details: http://en.wikipedia.org/wiki/List_of_moment_of_inertia_tensors
              m = 2.4 kg; h = 0.09 m; r = 0.175 m
@@ -679,10 +704,10 @@
     </link>
     <!-- Chaster wheel chassis3 -->
-    <joint name="chaster_wheel_chassis_joint3" type="revolute">
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