Commit message: first model descripiton pkg is uploaded

File: src/service_description/urdf/servicebot.urdf.xacro (robot description, xacro)
@@ -31,25 +31,4 @@
     <color rgba="0 1 0 1" />
   </material>
-  <material name="yellow">
-    <color rgba="1 1 0 1" />
-  </material>
-  <material name="grey">
-    <color rgba="0.5 0.5 0.5 1" />
-  </material>
-  <material name="orange">
-    <color rgba="1 0.5 0 1" />
-  </material>
-  <material name="brown">
-    <color rgba="0.5 0.25 0 1" />
-  </material>
-  <material name="purple">
-    <color rgba="0.5 0 0.5 1" />
-  </material>
-  <material name="cyan">
-    <color rgba="0 1 1 1" />
-  </material>
-  <material name="magenta">
-    <color rgba="1 0 1 1" />
-  </material>
   <!-- xacro material property -->
   <!-- servicebot -->
@@ -89,5 +68,5 @@
         <!-- COM experimentally determined -->
         <origin xyz="0.01 0 0" />
-        <mass value="20" /> <!--  kg for small/big battery pack -->
+        <mass value="15" /> <!--  kg for small/big battery pack -->
         <!-- servicebot's inertia tensor is approximated by a cylinder with homogeneous mass distribution
              More details: http://en.wikipedia.org/wiki/List_of_moment_of_inertia_tensors
@@ -236,5 +215,5 @@
       <!-- prismatic -->
       <!-- <origin xyz="0.07 -0.0765 0" rpy="1.5707 0 0 " /> -->
-      <origin xyz="0 -0.0765 -0.043" rpy="0 0 0 " />
+      <origin xyz="0 -0.0765 -0.04" rpy="0 0 0 " />
       <parent link="supan_pole2" />
       <child link="motor_baglanti_plaka" />
@@ -274,5 +253,5 @@
       <!-- prismatic -->
       <!-- <origin xyz="0.07 -0.0765 0" rpy="1.5707 0 0 " /> -->
-      <origin xyz="0 -0.0765 -0.043" rpy="0 0 0 " />
+      <origin xyz="0 -0.0765 -0.04" rpy="0 0 0 " />
       <parent link="supan_pole3" />
       <child link="motor_baglanti_plaka2" />
@@ -348,5 +327,5 @@
     <joint name="motor_joint2" type="fixed">
       <!-- prismatic -->
-      <origin xyz="0.02 0.0 -0.032" rpy="0 0 0" /> <!-- visual and collision, joint shift -->
+      <origin xyz="0.02 0.0 -0.03" rpy="0 0 0" /> <!-- visual and collision, joint shift -->
       <parent link="motor_baglanti_plaka2" />
       <child link="motor2" />
@@ -385,5 +364,5 @@
     <joint name="reduktor_mil_joint1" type="fixed">
       <!-- prismatic -->
-      <origin xyz="0.055 0.0 0.0" rpy="0 0 0" />
+      <origin xyz="0.058 0.0 0.0" rpy="0 0 0" />
       <parent link="motor1" />
       <child link="reduktor_mil1" />
@@ -394,5 +373,5 @@
       <visual>
         <geometry>
-          <mesh filename="package://service_description/meshes/servis/reduktor_mili.STL" scale="0.001 0.001 0.001" />
+          <mesh filename="package://service_description/meshes/servis/reduktor_mili.STL" scale="0.001 0.001 0.002" />
         </geometry>
         <origin xyz="-0.013 -0.007 0.007" rpy="0 1.57079 0" />
@@ -401,5 +380,5 @@
         <geometry>
           <!-- <cylinder length="0.142" radius="0.006" /> -->
-          <mesh filename="package://service_description/meshes/servis/reduktor_mili.STL" scale="0.001 0.001 0.001" />
+          <mesh filename="package://service_description/meshes/servis/reduktor_mili.STL" scale="0.001 0.001 0.002" />
         </geometry>
         <origin xyz="-0.013 -0.007 0.007" rpy="0 1.57079 0" />
@@ -421,5 +400,5 @@
     <!-- Reductor mil2 -->
     <joint name="reduktor_mil_joint2" type="fixed">
-      <origin xyz="-0.055 0.0 0.0" rpy="0 0 0" />
+      <origin xyz="-0.058 0.0 0.0" rpy="0 0 0" />
       <parent link="motor2" />
       <child link="reduktor_mil2" />
@@ -430,5 +409,5 @@
       <visual>
         <geometry>
-          <mesh filename="package://service_description/meshes/servis/reduktor_mili.STL" scale="0.001 0.001 0.001" />
+          <mesh filename="package://service_description/meshes/servis/reduktor_mili.STL" scale="0.001 0.001 0.002" />
         </geometry>
         <origin xyz="0.013 -0.007 -0.007" rpy="0 -1.57079 0" />
@@ -437,5 +416,5 @@
         <geometry>
           <!-- <cylinder length="0.142" radius="0.006" /> -->
-          <mesh filename="package://service_description/meshes/servis/reduktor_mili.STL" scale="0.001 0.001 0.001" />
+          <mesh filename="package://service_description/meshes/servis/reduktor_mili.STL" scale="0.001 0.001 0.002" />
         </geometry>
         <origin xyz="0.013 -0.007 -0.007" rpy="0 -1.57079 0" />
@@ -460,22 +439,21 @@
       <origin xyz="0.04 0.0 0.0" rpy="0 0 0" />
       <parent link="reduktor_mil1" />
-      <child link="reduktorteker1" />
+      <child link="reduktor1" />
       <axis xyz="1 0 0" />
       <!-- <limit lower="-0.15" upper="0.15" effort="100" velocity="0.01" /> -->
-      <limit effort="100" velocity="20" />
-    </joint>
-    <link name="reduktorteker1">
-      <visual>
-        <geometry>
-          <mesh filename="package://service_description/meshes/servis/reduktorteker.STL" scale="0.001 0.001 0.001" />
-        </geometry>
-        <origin xyz="-0.155 -0.079 ${0.0725 + 0.01}" rpy="0 1.57079 0" />
-      </visual>
-      <collision>
-        <geometry>
-          <!-- <cylinder length="0.142" radius="0.006" /> -->
-          <mesh filename="package://service_description/meshes/servis/reduktorteker.STL" scale="0.001 0.001 0.001" />
-        </geometry>
-        <origin xyz="-0.155 -0.079 ${0.0725 + 0.01}" rpy="0 1.57079 0" />
+    </joint>
+    <link name="reduktor1">
+      <visual>
+        <geometry>
+          <mesh filename="package://service_description/meshes/servis/reduktor.STL" scale="0.001 0.001 0.001" />
+        </geometry>
+        <origin xyz="-0.155 -0.0725 ${0.0725 + 0.01}" rpy="0 1.57079 0" />
+      </visual>
+      <collision>
+        <geometry>
+          <!-- <cylinder length="0.142" radius="0.006" /> -->
+          <mesh filename="package://service_description/meshes/servis/reduktor.STL" scale="0.001 0.001 0.001" />
+        </geometry>
+        <origin xyz="-0.155 -0.0725 ${0.0725 + 0.01}" rpy="0 1.57079 0" />
       </collision>
       <inertial>
@@ -497,20 +475,97 @@
       <origin xyz="-0.04 0.0 0.0" rpy="0 0 0" />
       <parent link="reduktor_mil2" />
-      <child link="reduktorteker2" />
+      <child link="reduktor2" />
       <axis xyz="1 0 0" />
       <!-- <limit lower="-0.15" upper="0.15" effort="100" velocity="0.01" /> -->
-      <limit effort="100" velocity="20" />
-    </joint>
-    <link name="reduktorteker2">
-      <visual>
-        <geometry>
-          <mesh filename="package://service_description/meshes/servis/reduktorteker.STL" scale="0.001 0.001 0.001" />
+    </joint>
+    <link name="reduktor2">
+      <visual>
+        <geometry>
+          <mesh filename="package://service_description/meshes/servis/reduktor.STL" scale="0.001 0.001 0.001" />
+        </geometry>
+        <origin xyz="0.155 -0.0725 -${0.0725 + 0.01}" rpy="0 -1.57079 0" />
+      </visual>
+      <collision>
+        <geometry>
+          <!-- <cylinder length="0.142" radius="0.006" /> -->
+          <mesh filename="package://service_description/meshes/servis/reduktor.STL" scale="0.001 0.001 0.001" />
+        </geometry>
+        <origin xyz="0.155 -0.0725 -${0.0725 + 0.01}" rpy="0 -1.57079 0" />
+      </collision>
+      <inertial>
+        <!-- COM experimentally determined -->
+        <origin xyz="0.05375 -0.00689  -0.1" />
+        <mass value="0.21" /> <!--  kg for small/big battery pack -->
+        <!-- servicebot's inertia tensor is approximated by a cylinder with homogeneous mass distribution
+             More details: http://en.wikipedia.org/wiki/List_of_moment_of_inertia_tensors
+             m = 2.4 kg; h = 0.09 m; r = 0.175 m
+             ixx = 1/12 * m * (3 * r^2 + h^2)
+             iyy = 1/12 * m * (3 * r^2 + h^2)
+             izz = 1/2 * m * r^2
+          -->
+        <inertia ixx="0.00057724" ixy="0.0" ixz="0.0" iyy="0.00057724" iyz="0.0" izz="0.00000597" />
+      </inertial>
+    </link>
+    <!-- Drive Wheel1 -->
+    <joint name="wheel_joint1" type="fixed">
+      <origin xyz="0.0 0.0 0.0" rpy="0 0 0" />
+      <parent link="reduktor1" />
+      <child link="wheel1" />
+      <!-- <axis xyz="0 1 0" /> -->
+      <!-- <limit lower="-0.15" upper="0.15" effort="100" velocity="0.01" /> -->
+    </joint>
+    <link name="wheel1">
+      <visual>
+        <geometry>
+          <mesh filename="package://service_description/meshes/servis/tahrik_tekeri.STL" scale="0.001 0.001 0.001" />
+        </geometry>
+        <origin xyz="-0.155 -0.079 ${0.0725 + 0.01}" rpy="0 1.57079 0" />
+      </visual>
+      <material name="green">
+        <color rgba="0 0 1 1" />
+      </material>
+      <collision>
+        <geometry>
+          <!-- <cylinder length="0.142" radius="0.006" /> -->
+          <mesh filename="package://service_description/meshes/servis/tahrik_tekeri.STL" scale="0.001 0.001 0.001" />
+        </geometry>
+        <origin xyz="-0.155 -0.079 ${0.0725 + 0.01}" rpy="0 1.57079 0" />
+      </collision>
+      <inertial>
+        <!-- COM experimentally determined -->
+        <origin xyz="0.05375 -0.00689  -0.1" />
+        <mass value="0.21" /> <!--  kg for small/big battery pack -->
+        <!-- servicebot's inertia tensor is approximated by a cylinder with homogeneous mass distribution
+             More details: http://en.wikipedia.org/wiki/List_of_moment_of_inertia_tensors
+             m = 2.4 kg; h = 0.09 m; r = 0.175 m
+             ixx = 1/12 * m * (3 * r^2 + h^2)
+             iyy = 1/12 * m * (3 * r^2 + h^2)
+             izz = 1/2 * m * r^2
+          -->
+        <inertia ixx="0.00057724" ixy="0.0" ixz="0.0" iyy="0.00057724" iyz="0.0" izz="0.00000597" />
+      </inertial>
+    </link>
+    <!-- Drive Wheel2 -->
+    <joint name="wheel_joint2" type="fixed">
+      <origin xyz="0.0 0.0 0.0" rpy="0 0 0" />
+      <parent link="reduktor2" />
+      <child link="wheel2" />
+      <!-- <axis xyz="0 1 0" /> -->
+      <!-- <limit lower="-0.15" upper="0.15" effort="100" velocity="0.01" /> -->
+    </joint>
+    <link name="wheel2">
+      <visual>
+        <geometry>
+          <mesh filename="package://service_description/meshes/servis/tahrik_tekeri.STL" scale="0.001 0.001 0.001" />
         </geometry>
         <origin xyz="0.155 -0.079 -${0.0725 + 0.01}" rpy="0 -1.57079 0" />
       </visual>
-      <collision>
-        <geometry>
-          <!-- <cylinder length="0.142" radius="0.006" /> -->
-          <mesh filename="package://service_description/meshes/servis/reduktorteker.STL" scale="0.001 0.001 0.001" />
+      <material name="green">
+        <color rgba="0 0 1 1" />
+      </material>
+      <collision>
+        <geometry>
+          <!-- <cylinder length="0.142" radius="0.006" /> -->
+          <mesh filename="package://service_description/meshes/servis/tahrik_tekeri.STL" scale="0.001 0.001 0.001" />
         </geometry>
         <origin xyz="0.155 -0.079 -${0.0725 + 0.01}" rpy="0 -1.57079 0" />
@@ -530,5 +585,4 @@
       </inertial>
     </link>
-    <!-- 3D camera -->
     <!-- Chaster wheel chassis1 -->
     <joint name="chaster_wheel_chassis_joint1" type="revolute">
@@ -537,6 +591,5 @@
       <child link="chaster_wheel_chassis1" />
       <axis xyz="0 0 1" />
-      <limit lower="3.14159" upper="3.14159" effort="10" velocity="1" />
-      <dynamics damping="0.01" friction="0.0" />
+      <limit lower="-3.1415926" upper="3.1415926" effort="100" velocity="0.1" />
     </joint>
     <link name="chaster_wheel_chassis1">
@@ -574,6 +627,5 @@
       <child link="chaster_wheel_chassis2" />
       <axis xyz="0 0 1" />
-      <limit lower="-3.14" upper="3.14" effort="10" velocity="1" />
-      <dynamics damping="0.01" friction="0.0" />
+      <limit lower="-3.1415926" upper="3.1415926" effort="100" velocity="0.1" />
     </joint>
     <link name="chaster_wheel_chassis2">
@@ -587,5 +639,5 @@
         <geometry>
           <!-- <cylinder length="0.142" radius="0.006" /> -->
-          <mesh filename="package://service_description/meshes/sarhos_tabla/sarhos_tabla.STL" scale="0.001 0.001 0.001" />
+          <mesh filename="package://service_description/meshes/servis/sarhos_tabla.STL" scale="0.001 0.001 0.001" />
         </geometry>
         <origin xyz="-0.03 0.03 -0.035" rpy="1.57079 0 0" />
@@ -611,6 +663,5 @@
       <child link="chaster_wheel_chassis3" />
       <axis xyz="0 0 1" />
-      <limit lower="-3.14" upper="3.14" effort="10" velocity="1" />
-      <dynamics damping="0.01" friction="0.0" />
+      <limit lower="-3.1415926" upper="3.1415926" effort="100" velocity="0.1" />
     </joint>
     <link name="chaster_wheel_chassis3">
@@ -648,5 +699,4 @@
       <child link="chaster_wheel1" />
       <axis xyz="1 0 0" />
-      <limit lower="-3.14" upper="3.14" effort="100" velocity="20" />
       <dynamics damping="0.1" friction="0.1" />
     </joint>
@@ -772,7 +822,4 @@
         </geometry>
         <origin xyz="-0.31 -0.32 -0.03" rpy="0 0 0" />
-        <material name="turquoise">
-          <color rgba="0 1 1 1" />
-        </material>
       </visual>
       <collision>
@@ -786,15 +833,42 @@
         <!-- COM experimentally determined -->
         <origin xyz="0.0 0.0 0.0" />
-        <mass value="30" /> <!--  kg for small/big battery pack -->
-        <!-- servicebot's inertia tensor is approximated by a cylinder with homogeneous mass distribution
-             More details: http://en.wikipedia.org/wiki/List_of_moment_of_inertia_tensors
-             m = 2.4 kg; h = 0.09 m; r = 0.175 m
-             ixx = 1/12 * m * (3 * r^2 + h^2)
-             iyy = 1/12 * m * (3 * r^2 + h^2)
-             izz = 1/2 * m * r^2
-          -->
-        <inertia ixx="0.0057724" ixy="0.0" ixz="0.0" iyy="0.0057724" iyz="0.0" izz="0.0000597" />
-      </inertial>
-    </link>
+        <mass value="0.20" /> <!--  kg for small/big battery pack -->
+        <!-- servicebot's inertia tensor is approximated by a cylinder with homogeneous mass distribution
+             More details: http://en.wikipedia.org/wiki/List_of_moment_of_inertia_tensors
+             m = 2.4 kg; h = 0.09 m; r = 0.175 m
+             ixx = 1/12 * m * (3 * r^2 + h^2)
+             iyy = 1/12 * m * (3 * r^2 + h^2)
+             izz = 1/2 * m * r^2
+          -->
+        <inertia ixx="0.00057724" ixy="0.0" ixz="0.0" iyy="0.00057724" iyz="0.0" izz="0.00000597" />
+      </inertial>
+    </link>
+    <!-- Rplidar-->
+    <link name="rplidar_laser_link">
+      <visual>
+        <origin rpy="0 0 ${2*M_PI_4}" xyz="0 0 0" />
+        <geometry>
+          <mesh filename="package://service_description/meshes/sensors/rplidar-a2.stl" />
+        </geometry>
+        <material name="dark_grey" />
+      </visual>
+      <collision>
+        <origin rpy="0 0 0" xyz="0 0 0" />
+        <geometry>
+          <cylinder length="0.01" radius="0.015" />
+        </geometry>
+      </collision>
+      <inertial>
+        <origin rpy="0 0 0" xyz="0 0 0" />
+        <mass value="0.1" />
+        <inertia ixx="6.458333333333333e-06" ixy="0" ixz="0" iyy="6.458333333333333e-06" iyz="0" izz="1.1249999999999999e-05" />
+      </inertial>
+    </link>
+    <joint name="rplidar_laser_joint" type="fixed">
+      <parent link="base_link" />
+      <child link="rplidar_laser_link" />
+      <origin rpy="0 0 0" xyz="0.0 0.18 0.25" />
+      <axis xyz="0 1 0" />
+    </joint>
     <!-- gazebo simulation plugin -->
     <xacro:servicebot_sim />

File: src/service_description/urdf/servicebot_gazebo.urdf.xacro (robot description, xacro)
@@ -2,72 +2,49 @@
 <robot name="servicebot_sim" xmlns:xacro="http://www.ros.org/wiki/xacro">
 	<xacro:macro name="servicebot_sim">
-		<gazebo reference="base_link">
-			<material>Gazebo/Blue</material>
-		</gazebo>
-		<gazebo reference="reduktorteker1">
-			<mu1 value="200.0" />
-			<mu2 value="100.0" />
-			<kp value="10000000.0" />
-			<kd value="1.0" />
+		<gazebo reference="reduktor1">
+			<mu1>1.0</mu1>
+			<mu2>1.0</mu2>
+			<kp>1000000.0</kp>
+			<kd>100.0</kd>
 			<minDepth>0.001</minDepth>
 			<maxVel>1.0</maxVel>
 			<maxForce>1000.0</maxForce>
-			<material>Gazebo/Green</material>
-			<turnGravityOff>false</turnGravityOff>
+			<material>Gazebo/Blue</material>
 		</gazebo>
-		<gazebo reference="reduktorteker2">
-			<mu1 value="200.0" />
-			<mu2 value="100.0" />
-			<kp value="10000000.0" />
-			<kd value="1.0" />
+		<gazebo reference="reduktor2">
+			<mu1>1.0</mu1>
+			<mu2>1.0</mu2>
+			<kp>1000000.0</kp>
+			<kd>100.0</kd>
 			<minDepth>0.001</minDepth>
 			<maxVel>1.0</maxVel>
-			<material>Gazebo/Green</material>
-			<turnGravityOff>false</turnGravityOff>
+			<material>Gazebo/Blue</material>
 		</gazebo>
 		<gazebo reference="chaster_wheel1">
-			<mu1 value="200.0" />
-			<mu2 value="100.0" />
-			<kp value="10000000.0" />
-			<kd value="1.0" />
+			<mu1>0.0</mu1>
+			<mu2>0.0</mu2>
+			<kp>1000000.0</kp>
+			<kd>100.0</kd>
 			<minDepth>0.001</minDepth>
 			<maxVel>1.0</maxVel>
-			<material>Gazebo/Green</material>
-			<turnGravityOff>false</turnGravityOff>
+			<material>Gazebo/FlatGray</material>
 		</gazebo>
 		<gazebo reference="chaster_wheel2">
-			<mu1 value="200.0" />
-			<mu2 value="100.0" />
-			<kp value="10000000.0" />
-			<kd value="1.0" />
+			<mu1>0.0</mu1>
+			<mu2>0.0</mu2>
+			<kp>1000000.0</kp>
+			<kd>100.0</kd>
 			<minDepth>0.001</minDepth>
 			<maxVel>1.0</maxVel>
-			<material>Gazebo/Green</material>
-			<turnGravityOff>false</turnGravityOff>
+			<material>Gazebo/FlatGray</material>
 		</gazebo>
 		<gazebo reference="chaster_wheel3">
-			<mu1 value="200.0" />
-			<mu2 value="100.0" />
-			<kp value="10000000.0" />
-			<kd value="1.0" />
+			<mu1>0.0</mu1>
+			<mu2>0.0</mu2>
+			<kp>1000000.0</kp>
+			<kd>100.0</kd>
 			<minDepth>0.001</minDepth>
 			<maxVel>1.0</maxVel>
-			<material>Gazebo/Green</material>
-			<turnGravityOff>false</turnGravityOff>
-		</gazebo>
-		<gazebo reference="upper_chassis">
-			<material>Gazebo/Turquoise</material>
-		</gazebo>
-		<gazebo reference="motor1">
-			<material>Gazebo/Red</material>
-		</gazebo>
-		<gazebo reference="motor2">
-			<material>Gazebo/Red</material>
-		</gazebo>
-		<gazebo reference="motor_baglanti_plaka">
-			<material>Gazebo/Yellow</material>
-		</gazebo>
-		<gazebo reference="motor_baglanti_plaka2">
-			<material>Gazebo/Yellow</material>
+			<material>Gazebo/FlatGray</material>
 		</gazebo>
 		<!-- This block connects the wheel joint to an actuator (motor), which informs both
@@ -76,8 +53,8 @@
 			<type>transmission_interface/SimpleTransmission</type>
 			<actuator name="wheel_motor2">
-				<mechanicalReduction>1</mechanicalReduction>
+				<mechanicalReduction>21</mechanicalReduction>
 			</actuator>
-			<joint name="reduktor_joint2">
-				<hardwareInterface>hardware_interface/VelocityJointInterface</hardwareInterface>
+			<joint name="$reduktor_joint2">
+				<hardwareInterface>VelocityJointInterface</hardwareInterface>
 			</joint>
 		</transmission>
@@ -85,39 +62,72 @@
 			<type>transmission_interface/SimpleTransmission</type>
 			<actuator name="wheel_motor1">
-				<mechanicalReduction>1</mechanicalReduction>
+				<mechanicalReduction>21</mechanicalReduction>
 			</actuator>
 			<joint name="reduktor_joint1">
-				<hardwareInterface>hardware_interface/VelocityJointInterface</hardwareInterface>
+				<hardwareInterface>VelocityJointInterface</hardwareInterface>
 			</joint>
 		</transmission>
 		<!-- Gazebo plugin for ROS Control -->
-		<!-- <gazebo>
+		<gazebo>
 			<plugin name="gazebo_ros_control" filename="libgazebo_ros_control.so">
 				<robotNamespace>/</robotNamespace>
 			</plugin>
-		</gazebo> -->
+		</gazebo>
+		<gazebo reference="rplidar_laser_link">
+			<material>Gazebo/Grey</material>
+		</gazebo>
+		<!-- rplidar gazebo references -->
+		<gazebo reference="rplidar_laser_link">
+			<!-- type is either gpu_laser or laser -->
+			<sensor name="head_rplidar_sensor" type="ray">
+				<pose>0 0 0 0 0 0</pose>
+				<visualize>true</visualize>
+				<update_rate>12</update_rate>
+				<ray>
+					<scan>
+						<horizontal>
+							<samples>360</samples>
+							<resolution>1</resolution>
+							<min_angle>-3.1415</min_angle>
+							<max_angle>3.1415</max_angle>
+						</horizontal>
+					</scan>
+					<range>
+						<min>0.12</min>
+						<max>12.0</max>
+						<resolution>0.01</resolution>
+					</range>
+					<noise>
+						<type>gaussian</type>
+						<!--Noise parameters based on published spec for Hokuyo laser
+               achieving "+-30mm" accuracy at range < 10m.  A mean of 0.0m and
+               stddev of 0.01m will put 99.7% of samples within 0.03m of the true
+               reading. -->
+						<mean>0.0</mean>
+						<stddev>0.01</stddev>
+					</noise>
+				</ray>
+				<!-- plugin_name is either libgazebo_ros_laser.so or libgazebo_ros_gpu_laser.so-->
+				<plugin filename="libgazebo_ros_laser.so" name="gazebo_ros_head_hokuyo_controller">
+					<topicName>/servicebot/scan</topicName>
+					<frameName>rplidar_laser_link</frameName>
+				</plugin>
+			</sensor>
+		</gazebo>
 		<gazebo>
-			<plugin filename="libgazebo_ros_diff_drive.so" name="differential_drive_controller">
+			<plugin name="differential_drive_controller" filename="libgazebo_ros_diff_drive.so">
 				<alwaysOn>true</alwaysOn>
 				<updateRate>20</updateRate>
-				<publishTf> true </publishTf>
-				<leftJoint>reduktor_joint1</leftJoint>
+				<leftJoint>reduktor_joint2</leftJoint>
 				<rightJoint>reduktor_joint2</rightJoint>
 				<wheelSeparation>.230</wheelSeparation>
 				<wheelDiameter>0.070</wheelDiameter>
-				<torque>5.0</torque>
-				<commandTopic>/cmd_vel</commandTopic>
-				<odometrySource>world</odometrySource> <!-- 'encoder' instead of 'world' is also possible -->
-				<odometryTopic>/odom</odometryTopic> <!-- relative/name ,  /global/name  -->
-				<odometryFrame>/odom</odometryFrame>
-				<robotBaseFrame>/base_footprint</robotBaseFrame>
-				<publishOdomTF> true </publishOdomTF>
+				<torque>1.0</torque>
+				<commandTopic>cmd_vel</commandTopic>
+				<odometryTopic>odom</odometryTopic>
+				<odometryFrame>odom</odometryFrame>
+				<robotBaseFrame>base_footprint</robotBaseFrame>
 				<publishWheelJointState>true</publishWheelJointState>
-				<!-- Set to true to publish transforms for the wheel links, defaults to false -->
-				<publishWheelTF>false</publishWheelTF>
-				<wheelAcceleration> 2.8 </wheelAcceleration>
-				<wheelTorque> 5.0 </wheelTorque>
 				<legacyMode>true</legacyMode>
-				<rosDebugLevel> Debug </rosDebugLevel> <!-- <rosDebugLevel>Debug</rosDebugLevel> -->
 			</plugin>
 		</gazebo>
