Commit message: all components rotate 90 degree

File: src/service_description/urdf/servicebot.urdf.xacro (robot description, xacro)
@@ -56,5 +56,5 @@
         </geometry>
         <material name="blue" />
-        <origin xyz="-0.237 -0.254  -0.281" rpy="0 0 0" />
+        <origin xyz="-0.254 0.237  -0.281" rpy="0 0 -${pi/2}" />
       </visual>
       <collision>
@@ -63,5 +63,5 @@
           <!-- <cylinder length="0.16" radius="0.26" /> -->
         </geometry>
-        <origin xyz="-0.237 -0.254  -0.281" rpy="0 0 0" />
+        <origin xyz="-0.254 0.237  -0.281" rpy="0 0 -${pi/2}" />
       </collision>
       <inertial>
@@ -80,5 +80,5 @@
     </link>
     <joint name="pole_suspan1_joint" type="fixed">
-      <origin xyz="-0.1455 -0.0765 ${0.142+0.0056}" rpy="0 0 0" />
+      <origin xyz="0.0765 -0.1455  ${0.142+0.0056}" rpy="0 0 0" />
       <parent link="base_link" />
       <child link="supan_pole1" />
@@ -113,5 +113,5 @@
     </link>
     <joint name="pole_suspan2_joint" type="fixed">
-      <origin xyz="0.1455 0.0765 ${0.142+0.0056}" rpy="0 0 0" />
+      <origin xyz="-0.0765 0.1455  ${0.142+0.0056}" rpy="0 0 0" />
       <parent link="base_link" />
       <child link="supan_pole2" />
@@ -146,5 +146,5 @@
     </link>
     <joint name="pole_suspan3_joint" type="fixed">
-      <origin xyz="-0.1455 0.0765 ${0.142+0.0056}" rpy="0 0 0" />
+      <origin xyz="-0.0765 -0.1455 ${0.142+0.0056}" rpy="0 0 0" />
       <parent link="base_link" />
       <child link="supan_pole3" />
@@ -179,5 +179,5 @@
     </link>
     <joint name="supan_pole4_joint" type="fixed">
-      <origin xyz="0.1455 -0.0765 ${0.142+0.0056}" rpy="0 0 0" />
+      <origin xyz="0.0765 0.1455 ${0.142+0.0056}" rpy="0 0 0" />
       <parent link="base_link" />
       <child link="supan_pole4" />
@@ -215,5 +215,5 @@
       <!-- prismatic -->
       <!-- <origin xyz="0.07 -0.0765 0" rpy="1.5707 0 0 " /> -->
-      <origin xyz="0 -0.0765 -0.04" rpy="0 0 0 " />
+      <origin xyz="0.0765 0.0 -0.04" rpy="0 0 ${M_PI_2}" />
       <parent link="supan_pole2" />
       <child link="motor_baglanti_plaka" />
@@ -253,5 +253,5 @@
       <!-- prismatic -->
       <!-- <origin xyz="0.07 -0.0765 0" rpy="1.5707 0 0 " /> -->
-      <origin xyz="0 -0.0765 -0.04" rpy="0 0 0 " />
+      <origin xyz="0.0765 -0.0 -0.04" rpy="0 0 ${M_PI_2}" />
       <parent link="supan_pole3" />
       <child link="motor_baglanti_plaka2" />
@@ -264,5 +264,5 @@
           <mesh filename="package://service_description/meshes/servis/motor_baglanti.STL" scale="0.001 0.001 0.001" />
         </geometry>
-        <origin xyz="0.015  -0.176 -0.086" rpy="1.5707 0 -3.1415926" />
+        <origin xyz="0.015  -0.176 -0.086" rpy="1.5707 0 ${-M_PI}" />
       </visual>
       <collision>
@@ -271,5 +271,5 @@
           <mesh filename="package://service_description/meshes/servis/motor_baglanti.STL" scale="0.001 0.001 0.001" />
         </geometry>
-        <origin xyz="0.015 -0.176 -0.086" rpy="1.5707 0 3.1415926" />
+        <origin xyz="0.015 -0.176 -0.086" rpy="1.5707 0 ${M_PI}" />
       </collision>
       <inertial>
@@ -301,5 +301,5 @@
           <mesh filename="package://service_description/meshes/servis/motor_kutusu.STL" scale="0.001 0.001 0.001" />
         </geometry>
-        <origin xyz="-0.04 -0.03 0.03" rpy="0 1.57079 0" />
+        <origin xyz="-0.04 -0.03 0.03" rpy="0 ${M_PI_2} 0" />
       </visual>
       <collision>
@@ -308,5 +308,5 @@
           <mesh filename="package://service_description/meshes/servis/motor_kutusu.STL" scale="0.001 0.001 0.001" />
         </geometry>
-        <origin xyz="-0.04 -0.03 0.03" rpy="0 1.57079 0" />
+        <origin xyz="-0.04 -0.03 0.03" rpy="0 ${M_PI_2} 0" />
       </collision>
       <inertial>
@@ -338,5 +338,5 @@
           <mesh filename="package://service_description/meshes/servis/motor_kutusu.STL" scale="0.001 0.001 0.001" />
         </geometry>
-        <origin xyz="0.04 -0.03 -0.03" rpy="0 -1.57079 0" />
+        <origin xyz="0.04 -0.03 -0.03" rpy="0 ${-M_PI_2} 0" />
       </visual>
       <collision>
@@ -345,5 +345,5 @@
           <mesh filename="package://service_description/meshes/servis/motor_kutusu.STL" scale="0.001 0.001 0.001" />
         </geometry>
-        <origin xyz="0.04 -0.03 -0.03" rpy="0 -1.57079 0" />
+        <origin xyz="0.04 -0.03 -0.03" rpy="0 ${-M_PI_2} 0" />
       </collision>
       <inertial>
@@ -375,5 +375,5 @@
           <mesh filename="package://service_description/meshes/servis/reduktor_mili.STL" scale="0.001 0.001 0.002" />
         </geometry>
-        <origin xyz="-0.013 -0.007 0.007" rpy="0 1.57079 0" />
+        <origin xyz="-0.013 -0.007 0.007" rpy="0 ${M_PI_2} 0" />
       </visual>
       <collision>
@@ -382,5 +382,5 @@
           <mesh filename="package://service_description/meshes/servis/reduktor_mili.STL" scale="0.001 0.001 0.002" />
         </geometry>
-        <origin xyz="-0.013 -0.007 0.007" rpy="0 1.57079 0" />
+        <origin xyz="-0.013 -0.007 0.007" rpy="0 ${M_PI_2} 0" />
       </collision>
       <inertial>
@@ -448,5 +448,5 @@
           <mesh filename="package://service_description/meshes/servis/reduktor.STL" scale="0.001 0.001 0.001" />
         </geometry>
-        <origin xyz="-0.155 -0.0725 ${0.0725 + 0.01}" rpy="0 1.57079 0" />
+        <origin xyz="-0.155 -0.0725 ${0.0725 + 0.01}" rpy="0 ${M_PI_2} 0" />
       </visual>
       <collision>
@@ -455,5 +455,5 @@
           <mesh filename="package://service_description/meshes/servis/reduktor.STL" scale="0.001 0.001 0.001" />
         </geometry>
-        <origin xyz="-0.155 -0.0725 ${0.0725 + 0.01}" rpy="0 1.57079 0" />
+        <origin xyz="-0.155 -0.0725 ${0.0725 + 0.01}" rpy="0 ${M_PI_2} 0" />
       </collision>
       <inertial>
@@ -484,5 +484,5 @@
           <mesh filename="package://service_description/meshes/servis/reduktor.STL" scale="0.001 0.001 0.001" />
         </geometry>
-        <origin xyz="0.155 -0.0725 -${0.0725 + 0.01}" rpy="0 -1.57079 0" />
+        <origin xyz="0.155 -0.0725 -${0.0725 + 0.01}" rpy="0 ${-M_PI_2} 0" />
       </visual>
       <collision>
@@ -491,5 +491,5 @@
           <mesh filename="package://service_description/meshes/servis/reduktor.STL" scale="0.001 0.001 0.001" />
         </geometry>
-        <origin xyz="0.155 -0.0725 -${0.0725 + 0.01}" rpy="0 -1.57079 0" />
+        <origin xyz="0.155 -0.0725 -${0.0725 + 0.01}" rpy="0 ${-M_PI_2} 0" />
       </collision>
       <inertial>
@@ -520,5 +520,5 @@
           <mesh filename="package://service_description/meshes/servis/tahrik_tekeri.STL" scale="0.001 0.001 0.001" />
         </geometry>
-        <origin xyz="-0.155 -0.079 ${0.0725 + 0.01}" rpy="0 1.57079 0" />
+        <origin xyz="-0.155 -0.079 ${0.0725 + 0.01}" rpy="0 ${M_PI_2} 0" />
       </visual>
       <material name="green">
@@ -530,5 +530,5 @@
           <mesh filename="package://service_description/meshes/servis/tahrik_tekeri.STL" scale="0.001 0.001 0.001" />
         </geometry>
-        <origin xyz="-0.155 -0.079 ${0.0725 + 0.01}" rpy="0 1.57079 0" />
+        <origin xyz="-0.155 -0.079 ${0.0725 + 0.01}" rpy="0 ${M_PI_2} 0" />
       </collision>
       <inertial>
@@ -559,5 +559,5 @@
           <mesh filename="package://service_description/meshes/servis/tahrik_tekeri.STL" scale="0.001 0.001 0.001" />
         </geometry>
-        <origin xyz="0.155 -0.079 -${0.0725 + 0.01}" rpy="0 -1.57079 0" />
+        <origin xyz="0.155 -0.079 -${0.0725 + 0.01}" rpy="0 ${-M_PI_2} 0" />
       </visual>
       <material name="green">
@@ -569,5 +569,5 @@
           <mesh filename="package://service_description/meshes/servis/tahrik_tekeri.STL" scale="0.001 0.001 0.001" />
         </geometry>
-        <origin xyz="0.155 -0.079 -${0.0725 + 0.01}" rpy="0 -1.57079 0" />
+        <origin xyz="0.155 -0.079 -${0.0725 + 0.01}" rpy="0 ${-M_PI_2} 0" />
       </collision>
       <inertial>
@@ -587,9 +587,9 @@
     <!-- Chaster wheel chassis1 -->
     <joint name="chaster_wheel_chassis_joint1" type="revolute">
-      <origin xyz="0.006 -0.198 0.047" rpy="0 0 0 " />
+      <origin xyz="-0.198 -0.01 0.047" rpy="0 0 0 " />
       <parent link="base_link" />
       <child link="chaster_wheel_chassis1" />
       <axis xyz="0 0 1" />
-      <limit lower="-3.1415926" upper="3.1415926" effort="100" velocity="0.1" />
+      <limit lower="${-M_PI}" upper="${M_PI}" effort="100" velocity="0.1" />
     </joint>
     <link name="chaster_wheel_chassis1">
@@ -598,5 +598,5 @@
           <mesh filename="package://service_description/meshes/sarhos_tabla/sarhos_tabla.STL" scale="0.001 0.001 0.001" />
         </geometry>
-        <origin xyz="-0.03 0.03 -0.035" rpy="1.57079 0 0" />
+        <origin xyz="-0.03 -0.03 -0.035" rpy="${M_PI_2} 0 ${M_PI_2}" />
       </visual>
       <collision>
@@ -605,5 +605,5 @@
           <mesh filename="package://service_description/meshes/sarhos_tabla/sarhos_tabla.STL" scale="0.001 0.001 0.001" />
         </geometry>
-        <origin xyz=" -0.03 0.03 -0.035" rpy="1.57079 0 0" />
+        <origin xyz=" -0.03 -0.03 -0.035" rpy="${M_PI_2} 0 ${M_PI_2}" />
       </collision>
       <inertial>
@@ -623,9 +623,9 @@
     <!-- Chaster wheel chassis2 -->
     <joint name="chaster_wheel_chassis_joint2" type="revolute">
-      <origin xyz="-0.115 0.156 0.047" rpy="0 0 0 " />
+      <origin xyz="0.156 -0.115 0.047" rpy="0 0 0 " />
       <parent link="base_link" />
       <child link="chaster_wheel_chassis2" />
       <axis xyz="0 0 1" />
-      <limit lower="-3.1415926" upper="3.1415926" effort="100" velocity="0.1" />
+      <limit lower="${-M_PI}" upper="${M_PI}" effort="100" velocity="0.1" />
     </joint>
     <link name="chaster_wheel_chassis2">
@@ -634,5 +634,5 @@
           <mesh filename="package://service_description/meshes/sarhos_tabla/sarhos_tabla.STL" scale="0.001 0.001 0.001" />
         </geometry>
-        <origin xyz="-0.03 0.03 -0.035" rpy="1.57079 0 0" />
+        <origin xyz="-0.03 -0.03 -0.035" rpy="${M_PI_2} 0 ${M_PI_2}" />
       </visual>
       <collision>
@@ -641,5 +641,5 @@
           <mesh filename="package://service_description/meshes/servis/sarhos_tabla.STL" scale="0.001 0.001 0.001" />
         </geometry>
-        <origin xyz="-0.03 0.03 -0.035" rpy="1.57079 0 0" />
+        <origin xyz="-0.03 -0.03 -0.035" rpy="${M_PI_2} 0 ${M_PI_2}" />
       </collision>
       <inertial>
@@ -659,9 +659,9 @@
     <!-- Chaster wheel chassis3 -->
     <joint name="chaster_wheel_chassis_joint3" type="revolute">
-      <origin xyz="0.115 0.156 0.047" rpy="0 0 0 " />
+      <origin xyz="0.156 0.115 0.047" rpy="0 0 0 " />
       <parent link="base_link" />
       <child link="chaster_wheel_chassis3" />
       <axis xyz="0 0 1" />
-      <limit lower="-3.1415926" upper="3.1415926" effort="100" velocity="0.1" />
+      <limit lower="${-M_PI}" upper="${M_PI}" effort="100" velocity="0.1" />
     </joint>
     <link name="chaster_wheel_chassis3">
@@ -670,5 +670,5 @@
           <mesh filename="package://service_description/meshes/sarhos_tabla/sarhos_tabla.STL" scale="0.001 0.001 0.001" />
         </geometry>
-        <origin xyz="-0.03 0.03 -0.035" rpy="1.57079 0 0" />
+        <origin xyz="-0.03 -0.03 -0.035" rpy="${M_PI_2} 0 ${M_PI_2}" />
       </visual>
       <collision>
@@ -677,5 +677,5 @@
           <mesh filename="package://service_description/meshes/sarhos_tabla/sarhos_tabla.STL" scale="0.001 0.001 0.001" />
         </geometry>
-        <origin xyz="-0.03 0.03 -0.035 " rpy="1.57079 0 0" />
+        <origin xyz="-0.03 -0.03 -0.035 " rpy="${M_PI_2} 0 ${M_PI_2}" />
       </collision>
       <inertial>
@@ -695,8 +695,8 @@
     <!-- chaster wheel1 -->
     <joint name="chaster_wheel_joint1" type="continuous">
-      <origin xyz="0.0 -0.025 -0.027" rpy="0 0 0 " />
+      <origin xyz="0.025 -0.0 -0.027" rpy="0 0 0 " />
       <parent link="chaster_wheel_chassis1" />
       <child link="chaster_wheel1" />
-      <axis xyz="1 0 0" />
+      <axis xyz="0 1 0" />
       <dynamics damping="0.1" friction="0.1" />
     </joint>
@@ -706,5 +706,5 @@
           <mesh filename="package://service_description/meshes/sarhos_tabla/sarhos_teker.STL" scale="0.001 0.001 0.001" />
         </geometry>
-        <origin xyz="-0.01 -0.025 -0.025" rpy="0 0 0" />
+        <origin xyz="-0.025 0.01 -0.025" rpy="0 0 ${-M_PI_2}" />
         <material name="green">
           <color rgba="0 1 0 1" />
@@ -716,5 +716,5 @@
           <mesh filename="package://service_description/meshes/sarhos_tabla/sarhos_teker.STL" scale="0.001 0.001 0.001" />
         </geometry>
-        <origin xyz="-0.01 -0.025 -0.025" rpy="0 0 0" />
+        <origin xyz="-0.025 0.01 -0.025" rpy="0 0 ${-M_PI_2}" />
       </collision>
       <inertial>
@@ -734,8 +734,8 @@
     <!-- chaster wheel2 -->
     <joint name="chaster_wheel_joint2" type="continuous">
-      <origin xyz="0.0 -0.025 -0.027" rpy="0 0 0 " />
+      <origin xyz="0.025 0.0 -0.027" rpy="0 0 0 " />
       <parent link="chaster_wheel_chassis2" />
       <child link="chaster_wheel2" />
-      <axis xyz="1 0 0" />
+      <axis xyz="0 1 0" />
       <dynamics damping="0.1" friction="0.1" />
     </joint>
@@ -745,5 +745,5 @@
           <mesh filename="package://service_description/meshes/sarhos_tabla/sarhos_teker.STL" scale="0.001 0.001 0.001" />
         </geometry>
-        <origin xyz="-0.01 -0.025 -0.025" rpy="0 0 0" />
+        <origin xyz="-0.025 0.01 -0.025" rpy="0 0 ${-M_PI_2}" />
         <material name="green">
           <color rgba="0 1 0 1" />
@@ -755,5 +755,5 @@
           <mesh filename="package://service_description/meshes/sarhos_tabla/sarhos_teker.STL" scale="0.001 0.001 0.001" />
         </geometry>
-        <origin xyz="-0.01 -0.025 -0.025" rpy="0 0 0" />
+        <origin xyz="-0.025 0.01 -0.025" rpy="0 0 ${-M_PI_2}" />
       </collision>
       <inertial>
@@ -773,8 +773,8 @@
     <!-- chaster wheel3 -->
     <joint name="chaster_wheel_joint3" type="continuous">
-      <origin xyz="0.0 -0.025 -0.027" rpy="0 0 0 " />
+      <origin xyz="0.025 0.0 -0.027" rpy="0 0 0 " />
       <parent link="chaster_wheel_chassis3" />
       <child link="chaster_wheel3" />
-      <axis xyz=" 1 0 0" />
+      <axis xyz=" 0 1 0" />
       <dynamics damping="0.1" friction="0.1" />
     </joint>
@@ -784,5 +784,5 @@
           <mesh filename="package://service_description/meshes/sarhos_tabla/sarhos_teker.STL" scale="0.001 0.001 0.001" />
         </geometry>
-        <origin xyz="-0.01 -0.025 -0.025" rpy="0 0 0" />
+        <origin xyz="-0.025 0.01 -0.025" rpy="0 0 ${-M_PI_2}" />
         <material name="green">
           <color rgba="0 1 0 1" />
@@ -794,5 +794,5 @@
           <mesh filename="package://service_description/meshes/sarhos_tabla/sarhos_teker.STL" scale="0.001 0.001 0.001" />
         </geometry>
-        <origin xyz="-0.01 -0.025 -0.025" rpy="0 0 0" />
+        <origin xyz="-0.025 0.01 -0.025" rpy="0 0 ${-M_PI_2}" />
       </collision>
       <inertial>
@@ -821,5 +821,5 @@
           <mesh filename="package://service_description/meshes/servis/ust_sase.STL" scale="0.001 0.001 0.001" />
         </geometry>
-        <origin xyz="-0.31 -0.32 -0.03" rpy="0 0 0" />
+        <origin xyz="-0.3 0.32 -0.03" rpy="0 0 -${pi/2}" />
       </visual>
       <collision>
@@ -828,5 +828,5 @@
           <mesh filename="package://service_description/meshes/servis/ust_sase.STL" scale="0.001 0.001 0.001" />
         </geometry>
-        <origin xyz="-0.31 -0.32 -0.03" rpy="0 0 0" />
+        <origin xyz="-0.3 0.32 -0.03" rpy="0 0 -${pi/2}" />
       </collision>
       <inertial>
@@ -868,6 +868,5 @@
       <parent link="base_link" />
       <child link="rplidar_laser_link" />
-      <origin rpy="0 0 0" xyz="0.0 0.18 0.25" />
-      <axis xyz="0 1 0" />
+      <origin rpy="0 0 -${2*M_PI_4}" xyz="0.18 0.0  0.25" />
     </joint>
     <!-- gazebo simulation plugin -->
