Commit message: all components rotate 90 degree

File: src/service_description/urdf/servicebot.urdf.xacro (robot description, xacro)
@@ -82,7 +82,7 @@
       <origin xyz="0.0765 -0.1455  ${0.142+0.0056}" rpy="0 0 0" />
       <parent link="base_link" />
-      <child link="supan_pole1" />
-    </joint>
-    <link name="supan_pole1">
+      <child link="suspan_pole1" />
+    </joint>
+    <link name="suspan_pole1">
       <visual>
         <geometry>
@@ -115,7 +115,7 @@
       <origin xyz="-0.0765 0.1455  ${0.142+0.0056}" rpy="0 0 0" />
       <parent link="base_link" />
-      <child link="supan_pole2" />
-    </joint>
-    <link name="supan_pole2">
+      <child link="suspan_pole2" />
+    </joint>
+    <link name="suspan_pole2">
       <visual>
         <geometry>
@@ -148,7 +148,7 @@
       <origin xyz="-0.0765 -0.1455 ${0.142+0.0056}" rpy="0 0 0" />
       <parent link="base_link" />
-      <child link="supan_pole3" />
-    </joint>
-    <link name="supan_pole3">
+      <child link="suspan_pole3" />
+    </joint>
+    <link name="suspan_pole3">
       <visual>
         <geometry>
@@ -178,10 +178,10 @@
       </inertial>
     </link>
-    <joint name="supan_pole4_joint" type="fixed">
+    <joint name="suspan_pole4_joint" type="fixed">
       <origin xyz="0.0765 0.1455 ${0.142+0.0056}" rpy="0 0 0" />
       <parent link="base_link" />
-      <child link="supan_pole4" />
-    </joint>
-    <link name="supan_pole4">
+      <child link="suspan_pole4" />
+    </joint>
+    <link name="suspan_pole4">
       <visual>
         <geometry>
@@ -216,5 +216,5 @@
       <!-- <origin xyz="0.07 -0.0765 0" rpy="1.5707 0 0 " /> -->
       <origin xyz="0.0765 0.0 -0.04" rpy="0 0 ${M_PI_2}" />
-      <parent link="supan_pole2" />
+      <parent link="suspan_pole2" />
       <child link="motor_baglanti_plaka" />
       <!-- <axis xyz="0 0 1" /> -->
@@ -254,5 +254,5 @@
       <!-- <origin xyz="0.07 -0.0765 0" rpy="1.5707 0 0 " /> -->
       <origin xyz="0.0765 -0.0 -0.04" rpy="0 0 ${M_PI_2}" />
-      <parent link="supan_pole3" />
+      <parent link="suspan_pole3" />
       <child link="motor_baglanti_plaka2" />
       <!-- <axis xyz="0 0.0 1" /> -->
@@ -290,5 +290,5 @@
     <joint name="motor_joint1" type="fixed">
       <!-- prismatic -->
-      <origin xyz="-0.02 0.0 -0.03" rpy="0 0 0" /> <!-- visual and collision, joint shift -->
+      <origin xyz="-0.02 0.0 -0.03" rpy="0 0 ${-M_PI_2}" /> <!-- visual and collision, joint shift -->
       <parent link="motor_baglanti_plaka" />
       <child link="motor1" />
@@ -301,5 +301,5 @@
           <mesh filename="package://service_description/meshes/servis/motor_kutusu.STL" scale="0.001 0.001 0.001" />
         </geometry>
-        <origin xyz="-0.04 -0.03 0.03" rpy="0 ${M_PI_2} 0" />
+        <origin xyz="0.03 -0.05 0.03" rpy="0 ${M_PI_2} ${M_PI_2}" />
       </visual>
       <collision>
@@ -308,5 +308,5 @@
           <mesh filename="package://service_description/meshes/servis/motor_kutusu.STL" scale="0.001 0.001 0.001" />
         </geometry>
-        <origin xyz="-0.04 -0.03 0.03" rpy="0 ${M_PI_2} 0" />
+        <origin xyz="0.03 -0.05 0.03" rpy="0 ${M_PI_2} ${M_PI_2}" />
       </collision>
       <inertial>
@@ -327,5 +327,5 @@
     <joint name="motor_joint2" type="fixed">
       <!-- prismatic -->
-      <origin xyz="0.02 0.0 -0.03" rpy="0 0 0" /> <!-- visual and collision, joint shift -->
+      <origin xyz="0.02 0.0 -0.03" rpy="0 0 ${-M_PI_2}" /> <!-- visual and collision, joint shift -->
       <parent link="motor_baglanti_plaka2" />
       <child link="motor2" />
@@ -338,5 +338,5 @@
           <mesh filename="package://service_description/meshes/servis/motor_kutusu.STL" scale="0.001 0.001 0.001" />
         </geometry>
-        <origin xyz="0.04 -0.03 -0.03" rpy="0 ${-M_PI_2} 0" />
+        <origin xyz="0.03 0.05 -0.03" rpy="0 ${-M_PI_2} ${M_PI_2}" />
       </visual>
       <collision>
@@ -345,5 +345,5 @@
           <mesh filename="package://service_description/meshes/servis/motor_kutusu.STL" scale="0.001 0.001 0.001" />
         </geometry>
-        <origin xyz="0.04 -0.03 -0.03" rpy="0 ${-M_PI_2} 0" />
+        <origin xyz="0.03 0.05 -0.03" rpy="0 ${-M_PI_2} ${M_PI_2}" />
       </collision>
       <inertial>
@@ -364,5 +364,5 @@
     <joint name="reduktor_mil_joint1" type="fixed">
       <!-- prismatic -->
-      <origin xyz="0.058 0.0 0.0" rpy="0 0 0" />
+      <origin xyz="0. 0.058 0.0" rpy="0 0 0" />
       <parent link="motor1" />
       <child link="reduktor_mil1" />
@@ -375,5 +375,5 @@
           <mesh filename="package://service_description/meshes/servis/reduktor_mili.STL" scale="0.001 0.001 0.002" />
         </geometry>
-        <origin xyz="-0.013 -0.007 0.007" rpy="0 ${M_PI_2} 0" />
+        <origin xyz="-0.007 0.013 0.007" rpy="0 ${M_PI_2} -${M_PI_2}" />
       </visual>
       <collision>
@@ -382,5 +382,5 @@
           <mesh filename="package://service_description/meshes/servis/reduktor_mili.STL" scale="0.001 0.001 0.002" />
         </geometry>
-        <origin xyz="-0.013 -0.007 0.007" rpy="0 ${M_PI_2} 0" />
+        <origin xyz="-0.007 -0.013 0.007" rpy="0 ${M_PI_2} -${M_PI_2}" />
       </collision>
       <inertial>
@@ -400,5 +400,5 @@
     <!-- Reductor mil2 -->
     <joint name="reduktor_mil_joint2" type="fixed">
-      <origin xyz="-0.058 0.0 0.0" rpy="0 0 0" />
+      <origin xyz="0. -0.058 0.0" rpy="0 0 0" />
       <parent link="motor2" />
       <child link="reduktor_mil2" />
@@ -411,5 +411,5 @@
           <mesh filename="package://service_description/meshes/servis/reduktor_mili.STL" scale="0.001 0.001 0.002" />
         </geometry>
-        <origin xyz="0.013 -0.007 -0.007" rpy="0 -1.57079 0" />
+        <origin xyz="-0.007 -0.013 -0.007" rpy="0 ${-M_PI_2} -${M_PI_2}" />
       </visual>
       <collision>
@@ -418,5 +418,5 @@
           <mesh filename="package://service_description/meshes/servis/reduktor_mili.STL" scale="0.001 0.001 0.002" />
         </geometry>
-        <origin xyz="0.013 -0.007 -0.007" rpy="0 -1.57079 0" />
+        <origin xyz="-0.007 -0.013 -0.007" rpy="0 ${M_PI_2} -${M_PI_2}" />
       </collision>
       <inertial>
@@ -437,8 +437,8 @@
     <joint name="reduktor_joint1" type="continuous">
       <!-- prismatic -->
-      <origin xyz="0.04 0.0 0.0" rpy="0 0 0" />
+      <origin xyz="0. 0.04 0.0" rpy="0 0 0" />
       <parent link="reduktor_mil1" />
       <child link="reduktor1" />
-      <axis xyz="1 0 0" />
+      <axis xyz="0 1 0" />
       <!-- <limit lower="-0.15" upper="0.15" effort="100" velocity="0.01" /> -->
     </joint>
@@ -448,5 +448,8 @@
           <mesh filename="package://service_description/meshes/servis/reduktor.STL" scale="0.001 0.001 0.001" />
         </geometry>
-        <origin xyz="-0.155 -0.0725 ${0.0725 + 0.01}" rpy="0 ${M_PI_2} 0" />
+        <origin xyz="0.0725 -0.155 ${0.0725 + 0.0105}" rpy="0 ${M_PI_2} ${M_PI_2}" />
+        <material name="bronze">
+          <color rgba="0.8 0.5 0.2 1.0" />
+        </material>
       </visual>
       <collision>
@@ -455,5 +458,5 @@
           <mesh filename="package://service_description/meshes/servis/reduktor.STL" scale="0.001 0.001 0.001" />
         </geometry>
-        <origin xyz="-0.155 -0.0725 ${0.0725 + 0.01}" rpy="0 ${M_PI_2} 0" />
+        <origin xyz="0.0725 -0.155 ${0.0725 + 0.0105}" rpy="0 ${M_PI_2} ${M_PI_2}" />
       </collision>
       <inertial>
@@ -473,8 +476,8 @@
     <!-- reduktor2 -->
     <joint name="reduktor_joint2" type="continuous">
-      <origin xyz="-0.04 0.0 0.0" rpy="0 0 0" />
+      <origin xyz="0.0 -0.04 0.0" rpy="0 0 0" />
       <parent link="reduktor_mil2" />
       <child link="reduktor2" />
-      <axis xyz="1 0 0" />
+      <axis xyz="0 1 0" />
       <!-- <limit lower="-0.15" upper="0.15" effort="100" velocity="0.01" /> -->
     </joint>
@@ -484,5 +487,8 @@
           <mesh filename="package://service_description/meshes/servis/reduktor.STL" scale="0.001 0.001 0.001" />
         </geometry>
-        <origin xyz="0.155 -0.0725 -${0.0725 + 0.01}" rpy="0 ${-M_PI_2} 0" />
+        <origin xyz="0.0725 0.155 -${0.0725 + 0.0095}" rpy="0 ${-M_PI_2} ${M_PI_2}" />
+        <material name="bronze">
+          <color rgba="0.8 0.5 0.2 1.0" />
+        </material>
       </visual>
       <collision>
@@ -491,5 +497,5 @@
           <mesh filename="package://service_description/meshes/servis/reduktor.STL" scale="0.001 0.001 0.001" />
         </geometry>
-        <origin xyz="0.155 -0.0725 -${0.0725 + 0.01}" rpy="0 ${-M_PI_2} 0" />
+        <origin xyz="0.0725 0.155 -${0.0725 + 0.0095}" rpy="0 ${-M_PI_2} ${M_PI_2}" />
       </collision>
       <inertial>
@@ -520,9 +526,9 @@
           <mesh filename="package://service_description/meshes/servis/tahrik_tekeri.STL" scale="0.001 0.001 0.001" />
         </geometry>
-        <origin xyz="-0.155 -0.079 ${0.0725 + 0.01}" rpy="0 ${M_PI_2} 0" />
-      </visual>
-      <material name="green">
-        <color rgba="0 0 1 1" />
-      </material>
+        <origin xyz="0.0785 -0.155 ${0.0725 + 0.0105}" rpy="0 ${M_PI_2} ${M_PI_2}" />
+        <material name="green">
+          <color rgba="0 0 1 1" />
+        </material>
+      </visual>
       <collision>
         <geometry>
@@ -530,5 +536,5 @@
           <mesh filename="package://service_description/meshes/servis/tahrik_tekeri.STL" scale="0.001 0.001 0.001" />
         </geometry>
-        <origin xyz="-0.155 -0.079 ${0.0725 + 0.01}" rpy="0 ${M_PI_2} 0" />
+        <origin xyz="0.0785 -0.155 ${0.0725 + 0.0105}" rpy="0 ${M_PI_2} ${M_PI_2}" />
       </collision>
       <inertial>
@@ -559,9 +565,9 @@
           <mesh filename="package://service_description/meshes/servis/tahrik_tekeri.STL" scale="0.001 0.001 0.001" />
         </geometry>
-        <origin xyz="0.155 -0.079 -${0.0725 + 0.01}" rpy="0 ${-M_PI_2} 0" />
-      </visual>
-      <material name="green">
-        <color rgba="0 0 1 1" />
-      </material>
+        <origin xyz="0.0785 0.155 -${0.0725 + 0.0095}" rpy="0 ${-M_PI_2} ${M_PI_2}" />
+        <material name="green">
+          <color rgba="0 0 1 1" />
+        </material>
+      </visual>
       <collision>
         <geometry>
@@ -569,5 +575,5 @@
           <mesh filename="package://service_description/meshes/servis/tahrik_tekeri.STL" scale="0.001 0.001 0.001" />
         </geometry>
-        <origin xyz="0.155 -0.079 -${0.0725 + 0.01}" rpy="0 ${-M_PI_2} 0" />
+        <origin xyz="0.0785 0.155 -${0.0725 + 0.0095}" rpy="0 ${-M_PI_2} ${M_PI_2}" />
       </collision>
       <inertial>
