Commit message: merge file is edited

File: src/service_description/urdf/service_library.urdf.xacro (robot description, xacro)
@@ -5,8 +5,8 @@
 <robot xmlns:xacro="http://www.ros.org/wiki/xacro">
   <!-- General -->
-  <xacro:include filename="$(find service_description)/urdf/common_properties.urdf.xacro" />
-  <xacro:include filename="$(find service_description)/urdf/servicebot_properties.urdf.xacro" />
+  <xacro:include filename="$(find service_description)/urdf/xacros/common_properties.urdf.xacro" />
+  <xacro:include filename="$(find service_description)/urdf/xacros/servicebot_properties.urdf.xacro" />
   <!-- Bases -->
-  <xacro:include filename="$(find service_description)/urdf/servicebot.urdf.xacro" />
+  <xacro:include filename="$(find service_description)/urdf/xacros/servicebot.urdf.xacro" />
   <!-- Stacks
     <xacro:include filename="$(find kobuki_description)/urdf/stacks/circles.urdf.xacro" />

File: src/service_description/urdf/servicebot.urdf.xacro (robot description, xacro)
@@ -7,6 +7,10 @@
  -->
 <robot name="servicebot" xmlns:xacro="http://www.ros.org/wiki/xacro">
-  <xacro:include filename="$(find service_description)/urdf/common_properties.urdf.xacro" />
-  <xacro:include filename="$(find service_description)/urdf/servicebot_gazebo.urdf.xacro" />
+  <xacro:include filename="$(find service_description)/urdf/xacros/common_properties.urdf.xacro" />
+  <xacro:include filename="$(find service_description)/urdf/xacros/servicebot_gazebo.urdf.xacro" />
+  <!-- Depth camera -->
+  <xacro:include filename="$(find service_description)/urdf/xacros/depth_camera.xacro" />
+  <!-- IMU -->
+  <xacro:include filename="$(find service_description)/urdf/xacros/imu.xacro" />
   <xacro:property name="width" value="0.2" />
   <xacro:property name="leglen" value="0.6" />
@@ -448,5 +452,5 @@
           <mesh filename="package://service_description/meshes/servis/reduktor.STL" scale="0.001 0.001 0.001" />
         </geometry>
-        <origin xyz="0.0725 -0.155 ${0.0725 + 0.0105}" rpy="0 ${M_PI_2} ${M_PI_2}" />
+        <origin xyz="0.0735 -0.155 ${0.0725 + 0.0099}" rpy="0 ${M_PI_2} ${M_PI_2}" />
         <material name="bronze">
           <color rgba="0.8 0.5 0.2 1.0" />
@@ -458,5 +462,5 @@
           <mesh filename="package://service_description/meshes/servis/reduktor.STL" scale="0.001 0.001 0.001" />
         </geometry>
-        <origin xyz="0.0725 -0.155 ${0.0725 + 0.0105}" rpy="0 ${M_PI_2} ${M_PI_2}" />
+        <origin xyz="0.0735 -0.155 ${0.0725 + 0.0099}" rpy="0 ${M_PI_2} ${M_PI_2}" />
       </collision>
       <inertial>
@@ -487,5 +491,5 @@
           <mesh filename="package://service_description/meshes/servis/reduktor.STL" scale="0.001 0.001 0.001" />
         </geometry>
-        <origin xyz="0.0725 0.155 -${0.0725 + 0.0095}" rpy="0 ${-M_PI_2} ${M_PI_2}" />
+        <origin xyz="0.0735 0.155 -${0.0725 + 0.0099}" rpy="0 ${-M_PI_2} ${M_PI_2}" />
         <material name="bronze">
           <color rgba="0.8 0.5 0.2 1.0" />
@@ -497,5 +501,5 @@
           <mesh filename="package://service_description/meshes/servis/reduktor.STL" scale="0.001 0.001 0.001" />
         </geometry>
-        <origin xyz="0.0725 0.155 -${0.0725 + 0.0095}" rpy="0 ${-M_PI_2} ${M_PI_2}" />
+        <origin xyz="0.0735 0.155 -${0.0725 + 0.0099}" rpy="0 ${-M_PI_2} ${M_PI_2}" />
       </collision>
       <inertial>
@@ -526,5 +530,5 @@
           <mesh filename="package://service_description/meshes/servis/tahrik_tekeri.STL" scale="0.001 0.001 0.001" />
         </geometry>
-        <origin xyz="0.0785 -0.155 ${0.0725 + 0.0105}" rpy="0 ${M_PI_2} ${M_PI_2}" />
+        <origin xyz="0.0798 -0.155 ${0.0725 + 0.0099}" rpy="0 ${M_PI_2} ${M_PI_2}" />
         <material name="green">
           <color rgba="0 0 1 1" />
@@ -536,5 +540,5 @@
           <mesh filename="package://service_description/meshes/servis/tahrik_tekeri.STL" scale="0.001 0.001 0.001" />
         </geometry>
-        <origin xyz="0.0785 -0.155 ${0.0725 + 0.0105}" rpy="0 ${M_PI_2} ${M_PI_2}" />
+        <origin xyz="0.0798 -0.155 ${0.0725 + 0.0099}" rpy="0 ${M_PI_2} ${M_PI_2}" />
       </collision>
       <inertial>
@@ -565,5 +569,5 @@
           <mesh filename="package://service_description/meshes/servis/tahrik_tekeri.STL" scale="0.001 0.001 0.001" />
         </geometry>
-        <origin xyz="0.0785 0.155 -${0.0725 + 0.0095}" rpy="0 ${-M_PI_2} ${M_PI_2}" />
+        <origin xyz="0.0798 0.155 -${0.0725 + 0.0099}" rpy="0 ${-M_PI_2} ${M_PI_2}" />
         <material name="green">
           <color rgba="0 0 1 1" />
@@ -575,5 +579,5 @@
           <mesh filename="package://service_description/meshes/servis/tahrik_tekeri.STL" scale="0.001 0.001 0.001" />
         </geometry>
-        <origin xyz="0.0785 0.155 -${0.0725 + 0.0095}" rpy="0 ${-M_PI_2} ${M_PI_2}" />
+        <origin xyz="0.0798 0.155 -${0.0725 + 0.0099}" rpy="0 ${-M_PI_2} ${M_PI_2}" />
       </collision>
       <inertial>
@@ -788,4 +792,5 @@
       <visual>
         <geometry>
+          <!-- <mesh filename="package://service_description/meshes/servis/ust_kaporta.STL" scale="0.001 0.001 0.001" /> -->
           <mesh filename="package://service_description/meshes/sarhos_tabla/sarhos_teker.STL" scale="0.001 0.001 0.001" />
         </geometry>
@@ -798,4 +803,5 @@
         <geometry>
           <!-- <cylinder length="0.142" radius="0.006" /> -->
+          <!-- <mesh filename="package://service_description/meshes/servis/ust_kaporta.STL" scale="0.001 0.001 0.001" /> -->
           <mesh filename="package://service_description/meshes/sarhos_tabla/sarhos_teker.STL" scale="0.001 0.001 0.001" />
         </geometry>
@@ -825,4 +831,5 @@
       <visual>
         <geometry>
+          <!-- <mesh filename="package://service_description/meshes/servis/ust_kaporta.STL" scale="0.001 0.001 0.001" /> -->
           <mesh filename="package://service_description/meshes/servis/ust_sase.STL" scale="0.001 0.001 0.001" />
         </geometry>
@@ -832,4 +839,5 @@
         <geometry>
           <!-- <cylinder length="0.142" radius="0.006" /> -->
+          <!-- <mesh filename="package://service_description/meshes/servis/ust_kaporta.STL" scale="0.001 0.001 0.001" /> -->
           <mesh filename="package://service_description/meshes/servis/ust_sase.STL" scale="0.001 0.001 0.001" />
         </geometry>
@@ -876,4 +884,16 @@
       <origin rpy="0 0 -${2*M_PI_4}" xyz="0.18 0.0  0.25" />
     </joint>
+    <!-- Depth Camera up-->
+    <xacro:depth_camera name="cameraup" parent="upper_chassis">
+      <origin xyz="0.228  -0.035   0.921" rpy="0 ${M_PI_4} 0" />
+    </xacro:depth_camera>
+    <!-- Depth Camera down-->
+    <xacro:depth_camera name="cameradown" parent="base_link">
+      <origin xyz="0.228 -0.035  0.094" rpy="0 -${M_PI_4} 0" />
+    </xacro:depth_camera>
+    <!-- imu -->
+    <xacro:imu name="imu" parent="base_link">
+      <origin xyz=" 0.128 0.02  0.19" rpy="0 0 0" />
+    </xacro:imu>
     <!-- gazebo simulation plugin -->
     <xacro:servicebot_sim />
