Commit message: refact: description pkg files edit

File: src/service_description/urdf/service_circle_a2_realsense.urdf.xacro (robot description, xacro)
@@ -4,5 +4,3 @@
     <!-- include the macro for the robot -->
     <xacro:servicebot />
-    <!-- <xacro:stack_hexagons parent="base_link" />
-    <xacro:sensor_kinect parent="base_link" /> -->
 </robot>

File: src/service_description/urdf/service_library.urdf.xacro (robot description, xacro)
@@ -9,10 +9,3 @@
   <!-- Bases -->
   <xacro:include filename="$(find service_description)/urdf/xacros/servicebot.urdf.xacro" />
-  <!-- Stacks
-    <xacro:include filename="$(find kobuki_description)/urdf/stacks/circles.urdf.xacro" />
-    <xacro:include filename="$(find kobuki_description)/urdf/stacks/hexagons.urdf.xacro" />
-  <xacro:include filename="$(find kobuki_description)/urdf/sensors/kinect.urdf.xacro" />
-  <xacro:include filename="$(find kobuki_description)/urdf/sensors/asus_xtion_pro.urdf.xacro" />
-  <xacro:include filename="$(find kobuki_description)/urdf/sensors/asus_xtion_pro_offset.urdf.xacro" />
-  -->
 </robot>

File: src/service_description/urdf/xacros/servicebot.urdf.xacro (robot description, xacro)
@@ -2,6 +2,7 @@
 <!--
   This is not a standalone urdf for servicebot. It simply defines the 'servicebot' tag that can
-  be incorporated by other urdf files (e.g. turtlebot).
-  See servicebot_standalone.urdf.xacro for a standalone urdf to be tested with
+be incorporated by other urdf files (e.g. turtlebot).
+  See servicebot_standalone.urdf.xacro for a
+standalone urdf to be tested with
       servicebot_description/launch/view_model.launch
  -->
@@ -20,8 +21,10 @@
     <!--
        Base link is set at the bottom of the base mould.
-       This is done to be compatible with the way base link
+       This is done to be
+    compatible with the way base link
        was configured for turtlebot 1. Refer to
-       https://github.com/turtlebot/turtlebot/issues/40
-       To put the base link at the more oft used wheel
+    https://github.com/turtlebot/turtlebot/issues/40
+       To put the base link at the more oft
+    used wheel
        axis, set the z-distance from the base_footprint
        to 0.352.
@@ -36,5 +39,6 @@
         <geometry>
           <!-- new mesh -->
-          <mesh filename="package://service_description/meshes/servis/sase2.STL" scale="0.001 0.001 0.001" />
+          <mesh filename="package://service_description/meshes/servis/sase2.STL"
+            scale="0.001 0.001 0.001" />
         </geometry>
         <material name="silver">
@@ -45,5 +49,6 @@
       <collision>
         <geometry>
-          <mesh filename="package://service_description/meshes/servis/sase2.STL" scale="0.001 0.001 0.001" />
+          <mesh filename="package://service_description/meshes/servis/sase2.STL"
+            scale="0.001 0.001 0.001" />
           <!-- <cylinder length="0.16" radius="0.26" /> -->
         </geometry>
@@ -54,9 +59,13 @@
         <origin xyz="0.01 0 0" />
         <mass value="15" /> <!--  kg for small/big battery pack -->
-        <!-- servicebot's inertia tensor is approximated by a cylinder with homogeneous mass distribution
-             More details: http://en.wikipedia.org/wiki/List_of_moment_of_inertia_tensors
-             m = 2.4 kg; h = 0.09 m; r = 0.175 m
-             ixx = 1/12 * m * (3 * r^2 + h^2)
-             iyy = 1/12 * m * (3 * r^2 + h^2)
+        <!-- servicebot's inertia tensor is approximated by a cylinder with homogeneous mass
+        distribution
+             More details:
+        http://en.wikipedia.org/wiki/List_of_moment_of_inertia_tensors
+             m = 2.4 kg; h =
+        0.09 m; r = 0.175 m
+             ixx = 1/12 * m * (3 * r^2 + h^2)
+             iyy = 1/12 *
+        m * (3 * r^2 + h^2)
              izz = 1/2 * m * r^2
           -->
@@ -72,5 +81,6 @@
       <visual>
         <geometry>
-          <mesh filename="package://service_description/meshes/servis/suspansiyon_mili.STL" scale="0.001 0.001 0.001" />
+          <mesh filename="package://service_description/meshes/servis/suspansiyon_mili.STL"
+            scale="0.001 0.001 0.001" />
         </geometry>
         <origin xyz="-0.006 -0.006 -0.071" rpy="0 0 0" />
@@ -79,5 +89,6 @@
         <geometry>
           <!-- <cylinder length="0.142" radius="0.006" /> -->
-          <mesh filename="package://service_description/meshes/servis/suspansiyon_mili.STL" scale="0.001 0.001 0.001" />
+          <mesh filename="package://service_description/meshes/servis/suspansiyon_mili.STL"
+            scale="0.001 0.001 0.001" />
         </geometry>
         <origin xyz="-0.006 -0.006 -0.071" rpy="0 0 0" />
@@ -87,9 +98,13 @@
         <origin xyz="0.1455 0.0765 0.141" />
         <mass value="0.21" /> <!--  kg for small/big battery pack -->
-        <!-- servicebot's inertia tensor is approximated by a cylinder with homogeneous mass distribution
-             More details: http://en.wikipedia.org/wiki/List_of_moment_of_inertia_tensors
-             m = 2.4 kg; h = 0.09 m; r = 0.175 m
-             ixx = 1/12 * m * (3 * r^2 + h^2)
-             iyy = 1/12 * m * (3 * r^2 + h^2)
+        <!-- servicebot's inertia tensor is approximated by a cylinder with homogeneous mass
+        distribution
+             More details:
+        http://en.wikipedia.org/wiki/List_of_moment_of_inertia_tensors
+             m = 2.4 kg; h =
+        0.09 m; r = 0.175 m
+             ixx = 1/12 * m * (3 * r^2 + h^2)
+             iyy = 1/12 *
+        m * (3 * r^2 + h^2)
              izz = 1/2 * m * r^2
           -->
@@ -105,5 +120,6 @@
       <visual>
         <geometry>
-          <mesh filename="package://service_description/meshes/servis/suspansiyon_mili.STL" scale="0.001 0.001 0.001" />
+          <mesh filename="package://service_description/meshes/servis/suspansiyon_mili.STL"
+            scale="0.001 0.001 0.001" />
         </geometry>
         <origin xyz="-0.006 -0.006 -0.071" rpy="0 0 0" />
@@ -112,5 +128,6 @@
         <geometry>
           <!-- <cylinder length="0.142" radius="0.006" /> -->
-          <mesh filename="package://service_description/meshes/servis/suspansiyon_mili.STL" scale="0.001 0.001 0.001" />
+          <mesh filename="package://service_description/meshes/servis/suspansiyon_mili.STL"
+            scale="0.001 0.001 0.001" />
         </geometry>
         <origin xyz="-0.006 -0.006 -0.071" rpy="0 0 0" />
@@ -120,9 +137,13 @@
         <origin xyz="-0.1455 -0.0765  0.141" />
         <mass value="0.21" /> <!--  kg for small/big battery pack -->
-        <!-- servicebot's inertia tensor is approximated by a cylinder with homogeneous mass distribution
-             More details: http://en.wikipedia.org/wiki/List_of_moment_of_inertia_tensors
-             m = 2.4 kg; h = 0.09 m; r = 0.175 m
-             ixx = 1/12 * m * (3 * r^2 + h^2)
-             iyy = 1/12 * m * (3 * r^2 + h^2)
+        <!-- servicebot's inertia tensor is approximated by a cylinder with homogeneous mass
+        distribution
+             More details:
+        http://en.wikipedia.org/wiki/List_of_moment_of_inertia_tensors
+             m = 2.4 kg; h =
+        0.09 m; r = 0.175 m
+             ixx = 1/12 * m * (3 * r^2 + h^2)
+             iyy = 1/12 *
+        m * (3 * r^2 + h^2)
              izz = 1/2 * m * r^2
           -->
@@ -138,5 +159,6 @@
       <visual>
         <geometry>
-          <mesh filename="package://service_description/meshes/servis/suspansiyon_mili.STL" scale="0.001 0.001 0.001" />
+          <mesh filename="package://service_description/meshes/servis/suspansiyon_mili.STL"
+            scale="0.001 0.001 0.001" />
         </geometry>
         <origin xyz="-0.006 -0.006 -0.071" rpy="0 0 0" />
@@ -145,5 +167,6 @@
         <geometry>
           <!-- <cylinder length="0.142" radius="0.006" /> -->
-          <mesh filename="package://service_description/meshes/servis/suspansiyon_mili.STL" scale="0.001 0.001 0.001" />
+          <mesh filename="package://service_description/meshes/servis/suspansiyon_mili.STL"
+            scale="0.001 0.001 0.001" />
         </geometry>
         <origin xyz="-0.006 -0.006 -0.071" rpy="0 0 0" />
@@ -153,9 +176,13 @@
         <origin xyz="-0.1455 0.0765 0.141" />
         <mass value="0.21" /> <!--  kg for small/big battery pack -->
-        <!-- servicebot's inertia tensor is approximated by a cylinder with homogeneous mass distribution
-             More details: http://en.wikipedia.org/wiki/List_of_moment_of_inertia_tensors
-             m = 2.4 kg; h = 0.09 m; r = 0.175 m
-             ixx = 1/12 * m * (3 * r^2 + h^2)
-             iyy = 1/12 * m * (3 * r^2 + h^2)
+        <!-- servicebot's inertia tensor is approximated by a cylinder with homogeneous mass
+        distribution
+             More details:
+        http://en.wikipedia.org/wiki/List_of_moment_of_inertia_tensors
+             m = 2.4 kg; h =
+        0.09 m; r = 0.175 m
+             ixx = 1/12 * m * (3 * r^2 + h^2)
+             iyy = 1/12 *
+        m * (3 * r^2 + h^2)
              izz = 1/2 * m * r^2
           -->
@@ -171,5 +198,6 @@
       <visual>
         <geometry>
-          <mesh filename="package://service_description/meshes/servis/suspansiyon_mili.STL" scale="0.001 0.001 0.001" />
+          <mesh filename="package://service_description/meshes/servis/suspansiyon_mili.STL"
+            scale="0.001 0.001 0.001" />
         </geometry>
         <origin xyz="-0.006 -0.006 -0.071" rpy="0 0 0" />
@@ -178,5 +206,6 @@
         <geometry>
           <!-- <cylinder length="0.142" radius="0.006" /> -->
-          <mesh filename="package://service_description/meshes/servis/suspansiyon_mili.STL" scale="0.001 0.001 0.001" />
+          <mesh filename="package://service_description/meshes/servis/suspansiyon_mili.STL"
+            scale="0.001 0.001 0.001" />
         </geometry>
         <origin xyz="-0.006 -0.006 -0.071" rpy="0 0 0" />
@@ -186,9 +215,13 @@
         <origin xyz="0.1455 -0.0765 0.141" />
         <mass value="0.21" /> <!--  kg for small/big battery pack -->
-        <!-- servicebot's inertia tensor is approximated by a cylinder with homogeneous mass distribution
-             More details: http://en.wikipedia.org/wiki/List_of_moment_of_inertia_tensors
-             m = 2.4 kg; h = 0.09 m; r = 0.175 m
-             ixx = 1/12 * m * (3 * r^2 + h^2)
-             iyy = 1/12 * m * (3 * r^2 + h^2)
+        <!-- servicebot's inertia tensor is approximated by a cylinder with homogeneous mass
+        distribution
+             More details:
+        http://en.wikipedia.org/wiki/List_of_moment_of_inertia_tensors
+             m = 2.4 kg; h =
+        0.09 m; r = 0.175 m
+             ixx = 1/12 * m * (3 * r^2 + h^2)
+             iyy = 1/12 *
+        m * (3 * r^2 + h^2)
              izz = 1/2 * m * r^2
           -->
@@ -209,5 +242,6 @@
       <visual>
         <geometry>
-          <mesh filename="package://service_description/meshes/servis/motor_baglanti.STL" scale="0.001 0.001 0.001" />
+          <mesh filename="package://service_description/meshes/servis/motor_baglanti.STL"
+            scale="0.001 0.001 0.001" />
         </geometry>
         <origin xyz="-0.015  0.176 -0.086" rpy="1.5707 0 0" />
@@ -216,5 +250,6 @@
         <geometry>
           <!-- <cylinder length="0.142" radius="0.006" /> -->
-          <mesh filename="package://service_description/meshes/servis/motor_baglanti.STL" scale="0.001 0.001 0.001" />
+          <mesh filename="package://service_description/meshes/servis/motor_baglanti.STL"
+            scale="0.001 0.001 0.001" />
         </geometry>
         <origin xyz="-0.015 0.176 -0.086" rpy="1.5707 0 0" />
@@ -224,9 +259,13 @@
         <origin xyz="0.05375 -0.00689  -0.1" />
         <mass value="0.21" /> <!--  kg for small/big battery pack -->
-        <!-- servicebot's inertia tensor is approximated by a cylinder with homogeneous mass distribution
-             More details: http://en.wikipedia.org/wiki/List_of_moment_of_inertia_tensors
-             m = 2.4 kg; h = 0.09 m; r = 0.175 m
-             ixx = 1/12 * m * (3 * r^2 + h^2)
-             iyy = 1/12 * m * (3 * r^2 + h^2)
+        <!-- servicebot's inertia tensor is approximated by a cylinder with homogeneous mass
+        distribution
+             More details:
+        http://en.wikipedia.org/wiki/List_of_moment_of_inertia_tensors
+             m = 2.4 kg; h =
+        0.09 m; r = 0.175 m
+             ixx = 1/12 * m * (3 * r^2 + h^2)
+             iyy = 1/12 *
+        m * (3 * r^2 + h^2)
              izz = 1/2 * m * r^2
           -->
@@ -247,5 +286,6 @@
       <visual>
         <geometry>
-          <mesh filename="package://service_description/meshes/servis/motor_baglanti.STL" scale="0.001 0.001 0.001" />
+          <mesh filename="package://service_description/meshes/servis/motor_baglanti.STL"
+            scale="0.001 0.001 0.001" />
         </geometry>
         <origin xyz="0.015  -0.176 -0.086" rpy="1.5707 0 ${-M_PI}" />
@@ -254,5 +294,6 @@
         <geometry>
           <!-- <cylinder length="0.142" radius="0.006" /> -->
-          <mesh filename="package://service_description/meshes/servis/motor_baglanti.STL" scale="0.001 0.001 0.001" />
+          <mesh filename="package://service_description/meshes/servis/motor_baglanti.STL"
+            scale="0.001 0.001 0.001" />
         </geometry>
         <origin xyz="0.015 -0.176 -0.086" rpy="1.5707 0 ${M_PI}" />
@@ -262,9 +303,13 @@
         <origin xyz="0.05375 -0.00689  -0.1" />
         <mass value="0.21" /> <!--  kg for small/big battery pack -->
-        <!-- servicebot's inertia tensor is approximated by a cylinder with homogeneous mass distribution
-             More details: http://en.wikipedia.org/wiki/List_of_moment_of_inertia_tensors
-             m = 2.4 kg; h = 0.09 m; r = 0.175 m
-             ixx = 1/12 * m * (3 * r^2 + h^2)
-             iyy = 1/12 * m * (3 * r^2 + h^2)
+        <!-- servicebot's inertia tensor is approximated by a cylinder with homogeneous mass
+        distribution
+             More details:
+        http://en.wikipedia.org/wiki/List_of_moment_of_inertia_tensors
+             m = 2.4 kg; h =
+        0.09 m; r = 0.175 m
+             ixx = 1/12 * m * (3 * r^2 + h^2)
+             iyy = 1/12 *
+        m * (3 * r^2 + h^2)
              izz = 1/2 * m * r^2
           -->
@@ -284,5 +329,6 @@
       <visual>
         <geometry>
-          <mesh filename="package://service_description/meshes/servis/motor_kutusu.STL" scale="0.001 0.001 0.001" />
+          <mesh filename="package://service_description/meshes/servis/motor_kutusu.STL"
+            scale="0.001 0.001 0.001" />
         </geometry>
         <origin xyz="0.03 -0.05 0.03" rpy="0 ${M_PI_2} ${M_PI_2}" />
@@ -291,5 +337,6 @@
         <geometry>
           <!-- <cylinder length="0.142" radius="0.006" /> -->
-          <mesh filename="package://service_description/meshes/servis/motor_kutusu.STL" scale="0.001 0.001 0.001" />
+          <mesh filename="package://service_description/meshes/servis/motor_kutusu.STL"
+            scale="0.001 0.001 0.001" />
         </geometry>
         <origin xyz="0.03 -0.05 0.03" rpy="0 ${M_PI_2} ${M_PI_2}" />
@@ -299,9 +346,13 @@
         <origin xyz="0.05375 -0.00689  -0.1" />
         <mass value="0.21" /> <!--  kg for small/big battery pack -->
-        <!-- servicebot's inertia tensor is approximated by a cylinder with homogeneous mass distribution
-             More details: http://en.wikipedia.org/wiki/List_of_moment_of_inertia_tensors
-             m = 2.4 kg; h = 0.09 m; r = 0.175 m
-             ixx = 1/12 * m * (3 * r^2 + h^2)
-             iyy = 1/12 * m * (3 * r^2 + h^2)
+        <!-- servicebot's inertia tensor is approximated by a cylinder with homogeneous mass
+        distribution
+             More details:
+        http://en.wikipedia.org/wiki/List_of_moment_of_inertia_tensors
+             m = 2.4 kg; h =
+        0.09 m; r = 0.175 m
+             ixx = 1/12 * m * (3 * r^2 + h^2)
+             iyy = 1/12 *
+        m * (3 * r^2 + h^2)
              izz = 1/2 * m * r^2
           -->
@@ -321,5 +372,6 @@
       <visual>
         <geometry>
-          <mesh filename="package://service_description/meshes/servis/motor_kutusu.STL" scale="0.001 0.001 0.001" />
+          <mesh filename="package://service_description/meshes/servis/motor_kutusu.STL"
+            scale="0.001 0.001 0.001" />
         </geometry>
         <origin xyz="0.03 0.05 -0.03" rpy="0 ${-M_PI_2} ${M_PI_2}" />
@@ -328,5 +380,6 @@
         <geometry>
           <!-- <cylinder length="0.142" radius="0.006" /> -->
-          <mesh filename="package://service_description/meshes/servis/motor_kutusu.STL" scale="0.001 0.001 0.001" />
+          <mesh filename="package://service_description/meshes/servis/motor_kutusu.STL"
+            scale="0.001 0.001 0.001" />
         </geometry>
         <origin xyz="0.03 0.05 -0.03" rpy="0 ${-M_PI_2} ${M_PI_2}" />
@@ -336,9 +389,13 @@
         <origin xyz="0.05375 -0.00689  -0.1" />
         <mass value="0.21" /> <!--  kg for small/big battery pack -->
-        <!-- servicebot's inertia tensor is approximated by a cylinder with homogeneous mass distribution
-             More details: http://en.wikipedia.org/wiki/List_of_moment_of_inertia_tensors
-             m = 2.4 kg; h = 0.09 m; r = 0.175 m
-             ixx = 1/12 * m * (3 * r^2 + h^2)
-             iyy = 1/12 * m * (3 * r^2 + h^2)
+        <!-- servicebot's inertia tensor is approximated by a cylinder with homogeneous mass
+        distribution
+             More details:
+        http://en.wikipedia.org/wiki/List_of_moment_of_inertia_tensors
+             m = 2.4 kg; h =
+        0.09 m; r = 0.175 m
+             ixx = 1/12 * m * (3 * r^2 + h^2)
+             iyy = 1/12 *
+        m * (3 * r^2 + h^2)
              izz = 1/2 * m * r^2
           -->
@@ -358,5 +415,6 @@
       <visual>
         <geometry>
-          <mesh filename="package://service_description/meshes/servis/reduktor_mili.STL" scale="0.001 0.001 0.002" />
+          <mesh filename="package://service_description/meshes/servis/reduktor_mili.STL"
+            scale="0.001 0.001 0.002" />
         </geometry>
         <origin xyz="-0.007 0.013 0.007" rpy="0 ${M_PI_2} -${M_PI_2}" />
@@ -365,5 +423,6 @@
         <geometry>
           <!-- <cylinder length="0.142" radius="0.006" /> -->
-          <mesh filename="package://service_description/meshes/servis/reduktor_mili.STL" scale="0.001 0.001 0.002" />
+          <mesh filename="package://service_description/meshes/servis/reduktor_mili.STL"
+            scale="0.001 0.001 0.002" />
         </geometry>
         <origin xyz="-0.007 0.013 0.007" rpy="0 ${M_PI_2} -${M_PI_2}" />
@@ -373,9 +432,13 @@
         <origin xyz="0.05375 -0.00689  -0.1" />
         <mass value="0.21" /> <!--  kg for small/big battery pack -->
-        <!-- servicebot's inertia tensor is approximated by a cylinder with homogeneous mass distribution
-             More details: http://en.wikipedia.org/wiki/List_of_moment_of_inertia_tensors
-             m = 2.4 kg; h = 0.09 m; r = 0.175 m
-             ixx = 1/12 * m * (3 * r^2 + h^2)
-             iyy = 1/12 * m * (3 * r^2 + h^2)
+        <!-- servicebot's inertia tensor is approximated by a cylinder with homogeneous mass
+        distribution
+             More details:
+        http://en.wikipedia.org/wiki/List_of_moment_of_inertia_tensors
+             m = 2.4 kg; h =
+        0.09 m; r = 0.175 m
+             ixx = 1/12 * m * (3 * r^2 + h^2)
+             iyy = 1/12 *
+        m * (3 * r^2 + h^2)
              izz = 1/2 * m * r^2
           -->
@@ -394,5 +457,6 @@
       <visual>
         <geometry>
-          <mesh filename="package://service_description/meshes/servis/reduktor_mili.STL" scale="0.001 0.001 0.002" />
+          <mesh filename="package://service_description/meshes/servis/reduktor_mili.STL"
+            scale="0.001 0.001 0.002" />
         </geometry>
         <origin xyz="-0.007 -0.013 -0.007" rpy="0 ${-M_PI_2} -${M_PI_2}" />
@@ -401,5 +465,6 @@
         <geometry>
           <!-- <cylinder length="0.142" radius="0.006" /> -->
-          <mesh filename="package://service_description/meshes/servis/reduktor_mili.STL" scale="0.001 0.001 0.002" />
+          <mesh filename="package://service_description/meshes/servis/reduktor_mili.STL"
+            scale="0.001 0.001 0.002" />
         </geometry>
         <origin xyz="-0.007 -0.013 -0.007" rpy="0 ${M_PI_2} -${M_PI_2}" />
@@ -409,9 +474,13 @@
         <origin xyz="0.05375 -0.00689  -0.1" />
         <mass value="0.21" /> <!--  kg for small/big battery pack -->
-        <!-- servicebot's inertia tensor is approximated by a cylinder with homogeneous mass distribution
-             More details: http://en.wikipedia.org/wiki/List_of_moment_of_inertia_tensors
-             m = 2.4 kg; h = 0.09 m; r = 0.175 m
-             ixx = 1/12 * m * (3 * r^2 + h^2)
-             iyy = 1/12 * m * (3 * r^2 + h^2)
+        <!-- servicebot's inertia tensor is approximated by a cylinder with homogeneous mass
+        distribution
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