Commit message: base anad lidar xacro file is added

File: src/service_description/urdf/xacro/servicebot.urdf.xacro (robot description, xacro)
@@ -13,4 +13,14 @@
   <!-- IMU -->
   <xacro:include filename="$(find service_description)/urdf/xacro/imu.xacro" />
+  <!-- Lidar -->
+  <xacro:include filename="$(find service_description)/urdf/xacro/lidar.xacro" />
+  <!-- Base -->
+  <xacro:include filename="$(find service_description)/urdf/xacro/base.xacro" />
+  <!-- Wheels -->
+  <xacro:include filename="$(find service_description)/urdf/xacro/wheels.xacro" />
+  <!-- Rplidar -->
+  <xacro:include filename="$(find service_description)/urdf/xacro/rplidar.xacro" />
+  <!-- Chasster wheel -->
+  <xacro:include filename="$(find service_description)/urdf/xacro/chasster_wheel.xacro" />
   <xacro:property name="width" value="0.2" />
   <xacro:property name="pi" value="3.1415" />
@@ -54,51 +64,9 @@
   <!-- servicebot -->
   <xacro:macro name="servicebot">
-    <link name="base_footprint" />
-    <!--
-       Base link is set at the bottom of the base mould.
-       This is done to be compatible with the way base link
-       was configured for turtlebot 1. Refer to
-       https://github.com/turtlebot/turtlebot/issues/40
-       To put the base link at the more oft used wheel
-       axis, set the z-distance from the base_footprint
-       to 0.352.
-      -->
-    <joint name="base_joint" type="fixed">
+    <!-- base_link -->
+    <xacro:base name="base_link" parent="base_footprint">
       <origin xyz="0 0 0.0302" rpy="0 0 0" />
-      <parent link="base_footprint" />
-      <child link="base_link" />
-    </joint>
-    <link name="base_link">
-      <visual>
-        <geometry>
-          <!-- new mesh -->
-          <mesh filename="package://service_description/meshes/servis/sase2.STL" scale="0.001 0.001 0.001" />
-        </geometry>
-        <material name="silver">
-          <color rgba="0.8 0.8 0.8 1.0" />
-        </material>
-        <origin xyz="-0.254 0.237  -0.281" rpy="0 0 -${pi/2}" />
-      </visual>
-      <collision>
-        <geometry>
-          <mesh filename="package://service_description/meshes/servis/sase2.STL" scale="0.001 0.001 0.001" />
-          <!-- <cylinder length="0.16" radius="0.26" /> -->
-        </geometry>
-        <origin xyz="-0.254 0.237  -0.281" rpy="0 0 -${pi/2}" />
-      </collision>
-      <inertial>
-        <!-- COM experimentally determined -->
-        <origin xyz="0.01 0 0" />
-        <mass value="15" /> <!--  kg for small/big battery pack -->
-        <!-- servicebot's inertia tensor is approximated by a cylinder with homogeneous mass distribution
-             More details: http://en.wikipedia.org/wiki/List_of_moment_of_inertia_tensors
-             m = 2.4 kg; h = 0.09 m; r = 0.175 m
-             ixx = 1/12 * m * (3 * r^2 + h^2)
-             iyy = 1/12 * m * (3 * r^2 + h^2)
-             izz = 1/2 * m * r^2
-          -->
-        <inertia ixx="0.37" ixy="0.0" ixz="0.0" iyy="0.28" iyz="0.0" izz="0.36" />
-      </inertial>
-    </link>
+    </xacro:base>
+    <!-- pole-suspan1 -->
     <joint name="pole_suspan1_joint" type="fixed">
       <origin xyz="0.0765 -0.1455  ${0.142+0.0056}" rpy="0 0 0" />
@@ -471,5 +439,5 @@
         </geometry>
         <!-- <origin xyz="-0.155 -0.079 ${0.0725 + 0.01}" rpy="0 1.5779 0" /> -->
-        <origin xyz="0.0735 -0.155 ${0.0725 + 0.0099}" rpy="0 ${M_PI_2} ${M_PI_2}" />
+        <origin xyz="0.079 -0.155 ${0.0725 + 0.0099}" rpy="0 ${M_PI_2} ${M_PI_2}" />
       </visual>
       <collision>
@@ -479,5 +447,5 @@
         </geometry>
         <!-- <origin xyz="-0.155 -0.079 ${0.0725 + 0.01}" rpy="0 1.57079 0" /> -->
-        <origin xyz="0.0735 -0.155 ${0.0725 + 0.0099}" rpy="0 ${M_PI_2} ${M_PI_2}" />
+        <origin xyz="0.079 -0.155 ${0.0725 + 0.0099}" rpy="0 ${M_PI_2} ${M_PI_2}" />
       </collision>
       <inertial>
@@ -512,5 +480,5 @@
         </geometry>
         <!-- <origin xyz="0.155 -0.079 -${0.0725 + 0.01}" rpy="0 -1.57079 0" /> -->
-        <origin xyz="0.0735 0.155 -${0.0725 + 0.0099}" rpy="0 ${-M_PI_2} ${M_PI_2}" />
+        <origin xyz="0.079 0.155 -${0.0725 + 0.0099}" rpy="0 ${-M_PI_2} ${M_PI_2}" />
       </visual>
       <collision>
@@ -520,5 +488,5 @@
         </geometry>
         <!-- <origin xyz="0.155 -0.079 -${0.0725 + 0.01}" rpy="0 -1.57079 0" /> -->
-        <origin xyz="0.0735 0.155 -${0.0725 + 0.0099}" rpy="0 ${-M_PI_2} ${M_PI_2}" />
+        <origin xyz="0.079 0.155 -${0.0725 + 0.0099}" rpy="0 ${-M_PI_2} ${M_PI_2}" />
       </collision>
       <inertial>
@@ -657,5 +625,4 @@
       </inertial>
     </link>
-    <!-- chaster wheel1 -->
     <joint name="chaster_wheel_joint1" type="continuous">
       <!-- <origin xyz="0.0 -0.025 -0.027" rpy="0 0 0 " /> -->
@@ -701,54 +668,12 @@
     </link>
     <!-- chaster wheel2 -->
-    <joint name="chaster_wheel_joint2" type="continuous">
+    <xacro:chaster_wheel name="chaster_wheel2" parent="chaster_wheel_chassis2" xyz="-0.025 0.01 -0.025" rpy="0 0 ${-M_PI_2}" >
       <!-- <origin xyz="0.0 -0.025 -0.027" rpy="0 0 0 " /> -->
       <origin xyz="0.025 0.0 -0.027" rpy="0 0 0 " />
-      <parent link="chaster_wheel_chassis2" />
-      <child link="chaster_wheel2" />
-      <axis xyz="0 1 0" />
-      <dynamics damping="0.1" friction="0.1" />
-    </joint>
-    <link name="chaster_wheel2">
-      <visual>
-        <geometry>
-          <mesh filename="package://service_description/meshes/sarhos_tabla/sarhos_teker.STL" scale="0.001 0.001 0.001" />
-        </geometry>
-        <!-- <origin xyz="-0.01 -0.025 -0.025" rpy="0 0 0" /> -->
-        <origin xyz="-0.025 0.01 -0.025" rpy="0 0 ${-M_PI_2}" />
-        <material name="green">
-          <color rgba="0 1 0 1" />
-        </material>
-      </visual>
-      <collision>
-        <geometry>
-          <!-- <cylinder length="0.142" radius="0.006" /> -->
-          <mesh filename="package://service_description/meshes/sarhos_tabla/sarhos_teker.STL" scale="0.001 0.001 0.001" />
-        </geometry>
-        <!-- <origin xyz="-0.01 -0.025 -0.025" rpy="0 0 0" /> -->
-        <origin xyz="-0.025 0.01 -0.025" rpy="0 0 ${-M_PI_2}" />
-      </collision>
-      <inertial>
-        <!-- COM experimentally determined -->
-        <origin xyz="0.0 0.0 0.0" />
-        <mass value="0.20" /> <!--  kg for small/big battery pack -->
-        <!-- servicebot's inertia tensor is approximated by a cylinder with homogeneous mass distribution
-             More details: http://en.wikipedia.org/wiki/List_of_moment_of_inertia_tensors
-             m = 2.4 kg; h = 0.09 m; r = 0.175 m
-             ixx = 1/12 * m * (3 * r^2 + h^2)
-             iyy = 1/12 * m * (3 * r^2 + h^2)
-             izz = 1/2 * m * r^2
-          -->
-        <inertia ixx="0.00057724" ixy="0.0" ixz="0.0" iyy="0.00057724" iyz="0.0" izz="0.00000597" />
-      </inertial>
-    </link>
+    </xacro:chaster_wheel>
     <!-- chaster wheel3 -->
-    <joint name="chaster_wheel_joint3" type="continuous">
-      <!-- <origin xyz="0.0 -0.025 -0.027" rpy="0 0 0 " /> -->
+    <xacro:chaster_wheel name="chaster_wheel3" parent="chaster_wheel_chassis3" xyz="0 0 0" rpy="0 0  ${2*M_PI_4}">
       <origin xyz="0.025 0.0 -0.027" rpy="0 0 0 " />
-      <parent link="chaster_wheel_chassis3" />
-      <child link="chaster_wheel3" />
-      <axis xyz=" 0 1 0" />
-      <dynamics damping="0.1" friction="0.1" />
-    </joint>
+    </xacro:chaster_wheel>
     <link name="chaster_wheel3">
       <visual>
@@ -825,31 +750,7 @@
     </link>
     <!-- Rplidar-->
-    <link name="rplidar_laser_link">
-      <visual>
-        <origin rpy="0 0 ${2*M_PI_4}" xyz="0 0 0" />
-        <geometry>
-          <mesh filename="package://service_description/meshes/sensors/rplidar-a2.stl" />
-        </geometry>
-        <material name="dark_grey">
-          <color rgba="0.2 0.2 0.2 1.0" />
-        </material>
-      </visual>
-      <collision>
-        <origin rpy="0 0 0" xyz="0 0 0" />
-        <geometry>
-          <cylinder length="0.01" radius="0.015" />
-        </geometry>
-      </collision>
-      <inertial>
-        <origin rpy="0 0 0" xyz="0 0 0" />
-        <mass value="0.1" />
-        <inertia ixx="6.458333333333333e-06" ixy="0" ixz="0" iyy="6.458333333333333e-06" iyz="0" izz="1.1249999999999999e-05" />
-      </inertial>
-    </link>
-    <joint name="rplidar_laser_joint" type="fixed">
-      <parent link="base_link" />
-      <child link="rplidar_laser_link" />
+    <xacro:rplidar name="rplidar" parent="base_link">
       <origin rpy="0 0 -${2*M_PI_4}" xyz="0.18 0.0  0.25" />
-    </joint>
+    </xacro:rplidar>
     <!-- Depth Camera up-->
     <xacro:depth_camera name="cameraup" parent="upper_chassis">

Commit message: wheel xacro file added and it is edited in base xacro file

File: src/service_description/urdf/xacro/servicebot.urdf.xacro (robot description, xacro)
@@ -625,88 +625,18 @@
       </inertial>
     </link>
-    <joint name="chaster_wheel_joint1" type="continuous">
+    <!-- Chaster wheel1 -->
+    <xacro:chasster_wheel name="chaster_wheel1" parent="chaster_wheel_chassis1" xyz="-0.025 0.01 -0.025" rpy="0 0 ${-M_PI_2}">
       <!-- <origin xyz="0.0 -0.025 -0.027" rpy="0 0 0 " /> -->
       <origin xyz="0.025 -0.0 -0.027" rpy="0 0 0 " />
-      <parent link="chaster_wheel_chassis1" />
-      <child link="chaster_wheel1" />
-      <!-- <axis xyz="1 0 0" /> -->
-      <axis xyz="0 1 0" />
-      <dynamics damping="0.1" friction="0.1" />
-    </joint>
-    <link name="chaster_wheel1">
-      <visual>
-        <geometry>
-          <mesh filename="package://service_description/meshes/sarhos_tabla/sarhos_teker.STL" scale="0.001 0.001 0.001" />
-        </geometry>
-        <!-- <origin xyz="-0.01 -0.025 -0.025" rpy="0 0 0" /> -->
-        <origin xyz="-0.025 0.01 -0.025" rpy="0 0 ${-M_PI_2}" />
-        <material name="green">
-          <color rgba="0 1 0 1" />
-        </material>
-      </visual>
-      <collision>
-        <geometry>
-          <!-- <cylinder length="0.142" radius="0.006" /> -->
-          <mesh filename="package://service_description/meshes/sarhos_tabla/sarhos_teker.STL" scale="0.001 0.001 0.001" />
-        </geometry>
-        <!-- <origin xyz="-0.01 -0.025 -0.025" rpy="0 0 0" /> -->
-        <origin xyz="-0.025 0.01 -0.025" rpy="0 0 ${-M_PI_2}" />
-      </collision>
-      <inertial>
-        <!-- COM experimentally determined -->
-        <origin xyz="0.0 0.0 0.0" />
-        <mass value="0.20" /> <!--  kg for small/big battery pack -->
-        <!-- servicebot's inertia tensor is approximated by a cylinder with homogeneous mass distribution
-             More details: http://en.wikipedia.org/wiki/List_of_moment_of_inertia_tensors
-             m = 2.4 kg; h = 0.09 m; r = 0.175 m
-             ixx = 1/12 * m * (3 * r^2 + h^2)
-             iyy = 1/12 * m * (3 * r^2 + h^2)
-             izz = 1/2 * m * r^2
-          -->
-        <inertia ixx="0.00057724" ixy="0.0" ixz="0.0" iyy="0.00057724" iyz="0.0" izz="0.00000597" />
-      </inertial>
-    </link>
+    </xacro:chasster_wheel>
     <!-- chaster wheel2 -->
-    <xacro:chaster_wheel name="chaster_wheel2" parent="chaster_wheel_chassis2" xyz="-0.025 0.01 -0.025" rpy="0 0 ${-M_PI_2}" >
+    <xacro:chaster_wheel name="chaster_wheel2" parent="chaster_wheel_chassis2" xyz="-0.025 0.01 -0.025" rpy="0 0 ${-M_PI_2}">
       <!-- <origin xyz="0.0 -0.025 -0.027" rpy="0 0 0 " /> -->
       <origin xyz="0.025 0.0 -0.027" rpy="0 0 0 " />
     </xacro:chaster_wheel>
     <!-- chaster wheel3 -->
-    <xacro:chaster_wheel name="chaster_wheel3" parent="chaster_wheel_chassis3" xyz="0 0 0" rpy="0 0  ${2*M_PI_4}">
+    <xacro:chaster_wheel name="chaster_wheel3" parent="chaster_wheel_chassis3" xyz="-0.025 0.01 -0.025" rpy="0 0 ${-M_PI_2}">
       <origin xyz="0.025 0.0 -0.027" rpy="0 0 0 " />
     </xacro:chaster_wheel>
-    <link name="chaster_wheel3">
-      <visual>
-        <geometry>
-          <mesh filename="package://service_description/meshes/sarhos_tabla/sarhos_teker.STL" scale="0.001 0.001 0.001" />
-        </geometry>
-        <!-- <origin xyz="-0.01 -0.025 -0.025" rpy="0 0 0" /> -->
-        <origin xyz="-0.025 0.01 -0.025" rpy="0 0 ${-M_PI_2}" />
-        <material name="green">
-          <color rgba="0 1 0 1" />
-        </material>
-      </visual>
-      <collision>
-        <geometry>
-          <!-- <cylinder length="0.142" radius="0.006" /> -->
-          <mesh filename="package://service_description/meshes/sarhos_tabla/sarhos_teker.STL" scale="0.001 0.001 0.001" />
-        </geometry>
-        <!-- <origin xyz="-0.01 -0.025 -0.025" rpy="0 0 0" /> -->
-        <origin xyz="-0.025 0.01 -0.025" rpy="0 0 ${-M_PI_2}" />
-      </collision>
-      <inertial>
-        <!-- COM experimentally determined -->
-        <origin xyz="0.0 0.0 0.0" />
-        <mass value="0.20" /> <!--  kg for small/big battery pack -->
-        <!-- servicebot's inertia tensor is approximated by a cylinder with homogeneous mass distribution
-             More details: http://en.wikipedia.org/wiki/List_of_moment_of_inertia_tensors
-             m = 2.4 kg; h = 0.09 m; r = 0.175 m
-             ixx = 1/12 * m * (3 * r^2 + h^2)
-             iyy = 1/12 * m * (3 * r^2 + h^2)
-             izz = 1/2 * m * r^2
-          -->
-        <inertia ixx="0.00057724" ixy="0.0" ixz="0.0" iyy="0.00057724" iyz="0.0" izz="0.00000597" />
-      </inertial>
-    </link>
     <!-- upper chassis -->
     <joint name="upper_chassis_joint" type="fixed">
