Commit message: refactor: REAL ROBOT URDF İS EDİT

File: src/service_description/urdf/xacro/base.xacro (robot description, xacro)
@@ -34,17 +34,4 @@
                 <origin xyz="-0.254 0.237  -0.281" rpy="0 0 -${pi/2}" />
             </collision>
-            <inertial>
-                <!-- COM experimentally determined -->
-                <origin xyz="0.0 0 0" />
-                <mass value="5" /> <!--  kg for small/big battery pack -->
-                <!-- servicebot's inertia tensor is approximated by a cylinder with homogeneous mass distribution
-             More details: http://en.wikipedia.org/wiki/List_of_moment_of_inertia_tensors
-             m = 2.4 kg; h = 0.09 m; r = 0.175 m
-             ixx = 1/12 * m * (3 * r^2 + h^2)
-             iyy = 1/12 * m * (3 * r^2 + h^2)
-             izz = 1/2 * m * r^2
-          -->
-                <inertia ixx="0.37" ixy="0.0" ixz="0.0" iyy="0.28" iyz="0.0" izz="0.36" />
-            </inertial>
         </link>
     </xacro:macro>

File: src/service_description/urdf/xacro/chasster_wheel.xacro (robot description, xacro)
@@ -18,18 +18,4 @@
                 </geometry>
             </collision>
-            <inertial>
-                <origin rpy="${rpy}" xyz="${xyz}" />
-                <mass value="0.1" />
-                <inertia ixx="6.458333333333333e-06" ixy="0" ixz="0" iyy="6.458333333333333e-06" iyz="0" izz="1.1249999999999999e-05">
-                    <!--  kg for small/big battery pack -->
-                    <!-- servicebot's inertia tensor is approximated by a cylinder with homogeneous mass distribution
-             More details: http://en.wikipedia.org/wiki/List_of_moment_of_inertia_tensors
-             m = 2.4 kg; h = 0.09 m; r = 0.175 m
-             ixx = 1/12 * m * (3 * r^2 + h^2)
-             iyy = 1/12 * m * (3 * r^2 + h^2)
-             izz = 1/2 * m * r^2
-          -->
-                </inertia>
-            </inertial>
         </link>
         <joint name="${name}_joint" type="continuous">
@@ -38,5 +24,4 @@
             <xacro:insert_block name="origin" />
             <axis xyz="0 1 0" />
-            <dynamics damping="0.1" friction="0.1" />
         </joint>
     </xacro:macro>

File: src/service_description/urdf/xacro/depth_camera.xacro (robot description, xacro)
@@ -17,5 +17,5 @@
 			<origin xyz="0 0.015 0" rpy="0 0 0" />
 			<parent link="${name}_link" />
-			<child link="${name}_link_gazebo" />
+			<child link="${name}_link_depth" />
 		</joint>
 		<link name="${name}_link">
@@ -35,12 +35,7 @@
 				</material>
 			</visual>
-			<inertial>
-				<mass value="1e-5" />
-				<origin xyz="0 0 0" rpy="0 0 0" />
-				<inertia ixx="1e-6" ixy="0" ixz="0" iyy="1e-6" iyz="0" izz="1e-6" />
-			</inertial>
 		</link>
 		<link name="${name}_link_optical"></link>
-		<link name="${name}_link_gazebo" />
+		<link name="${name}_link_depth" />
 	</xacro:macro>
 </robot>

File: src/service_description/urdf/xacro/imu.xacro (robot description, xacro)
@@ -17,9 +17,4 @@
         </material>
       </visual>
-      <inertial>
-        <mass value="0.001" />
-        <origin xyz="0 0 0" rpy="0 0 0" />
-        <inertia ixx="0.0001" ixy="0" ixz="0" iyy="0.000001" iyz="0" izz="0.0001" />
-      </inertial>
     </link>
   </xacro:macro>

File: src/service_description/urdf/xacro/rplidar.xacro (robot description, xacro)
@@ -18,9 +18,4 @@
                 </geometry>
             </collision>
-            <inertial>
-                <origin rpy="0 0 0" xyz="0 0 0" />
-                <mass value="0.1" />
-                <inertia ixx="6.458333333333333e-06" ixy="0" ixz="0" iyy="6.458333333333333e-06" iyz="0" izz="1.1249999999999999e-05" />
-            </inertial>
         </link>
         <joint name="rplidar_laser_joint" type="fixed">

File: src/service_description/urdf/xacro/servicebot.urdf.xacro (robot description, xacro)
@@ -8,5 +8,4 @@
 <robot name="servicebot" xmlns:xacro="http://www.ros.org/wiki/xacro">
   <xacro:include filename="$(find service_description)/urdf/xacro/common_properties.urdf.xacro" />
-  <xacro:include filename="$(find service_description)/urdf/xacro/servicebot_gazebo.urdf.xacro" />
   <!-- Depth camera -->
   <xacro:include filename="$(find service_description)/urdf/xacro/depth_camera.xacro" />
@@ -86,17 +85,4 @@
         <origin xyz="-0.006 -0.006 -0.071" rpy="0 0 0" />
       </collision>
-      <inertial>
-        <!-- COM experimentally determined -->
-        <origin xyz="0.1455 0.0765 0.141" />
-        <mass value="0.21" /> <!--  kg for small/big battery pack -->
-        <!-- servicebot's inertia tensor is approximated by a cylinder with homogeneous mass distribution
-             More details: http://en.wikipedia.org/wiki/List_of_moment_of_inertia_tensors
-             m = 2.4 kg; h = 0.09 m; r = 0.175 m
-             ixx = 1/12 * m * (3 * r^2 + h^2)
-             iyy = 1/12 * m * (3 * r^2 + h^2)
-             izz = 1/2 * m * r^2
-          -->
-        <inertia ixx="0.00057724" ixy="0.0" ixz="0.0" iyy="0.00057724" iyz="0.0" izz="0.00000597" />
-      </inertial>
     </link>
     <joint name="pole_suspan2_joint" type="fixed">
@@ -119,17 +105,4 @@
         <origin xyz="-0.006 -0.006 -0.071" rpy="0 0 0" />
       </collision>
-      <inertial>
-        <!-- COM experimentally determined -->
-        <origin xyz="-0.1455 -0.0765  0.141" />
-        <mass value="0.21" /> <!--  kg for small/big battery pack -->
-        <!-- servicebot's inertia tensor is approximated by a cylinder with homogeneous mass distribution
-             More details: http://en.wikipedia.org/wiki/List_of_moment_of_inertia_tensors
-             m = 2.4 kg; h = 0.09 m; r = 0.175 m
-             ixx = 1/12 * m * (3 * r^2 + h^2)
-             iyy = 1/12 * m * (3 * r^2 + h^2)
-             izz = 1/2 * m * r^2
-          -->
-        <inertia ixx="0.00057724" ixy="0.0" ixz="0.0" iyy="0.00057724" iyz="0.0" izz="0.00000597" />
-      </inertial>
     </link>
     <joint name="pole_suspan3_joint" type="fixed">
@@ -152,17 +125,4 @@
         <origin xyz="-0.006 -0.006 -0.071" rpy="0 0 0" />
       </collision>
-      <inertial>
-        <!-- COM experimentally determined -->
-        <origin xyz="-0.1455 0.0765 0.141" />
-        <mass value="0.21" /> <!--  kg for small/big battery pack -->
-        <!-- servicebot's inertia tensor is approximated by a cylinder with homogeneous mass distribution
-             More details: http://en.wikipedia.org/wiki/List_of_moment_of_inertia_tensors
-             m = 2.4 kg; h = 0.09 m; r = 0.175 m
-             ixx = 1/12 * m * (3 * r^2 + h^2)
-             iyy = 1/12 * m * (3 * r^2 + h^2)
-             izz = 1/2 * m * r^2
-          -->
-        <inertia ixx="0.00057724" ixy="0.0" ixz="0.0" iyy="0.00057724" iyz="0.0" izz="0.00000597" />
-      </inertial>
     </link>
     <joint name="suspan_pole4_joint" type="fixed">
@@ -185,17 +145,4 @@
         <origin xyz="-0.006 -0.006 -0.071" rpy="0 0 0" />
       </collision>
-      <inertial>
-        <!-- COM experimentally determined -->
-        <origin xyz="0.1455 -0.0765 0.141" />
-        <mass value="0.21" /> <!--  kg for small/big battery pack -->
-        <!-- servicebot's inertia tensor is approximated by a cylinder with homogeneous mass distribution
-             More details: http://en.wikipedia.org/wiki/List_of_moment_of_inertia_tensors
-             m = 2.4 kg; h = 0.09 m; r = 0.175 m
-             ixx = 1/12 * m * (3 * r^2 + h^2)
-             iyy = 1/12 * m * (3 * r^2 + h^2)
-             izz = 1/2 * m * r^2
-          -->
-        <inertia ixx="0.00057724" ixy="0.0" ixz="0.0" iyy="0.00057724" iyz="0.0" izz="0.00000597" />
-      </inertial>
     </link>
     <!-- Motor baglantı plakası1 -->
@@ -223,17 +170,4 @@
         <origin xyz="-0.015 0.176 -0.086" rpy="1.5707 0 0" />
       </collision>
-      <inertial>
-        <!-- COM experimentally determined -->
-        <origin xyz="0.05375 -0.00689  -0.1" />
-        <mass value="0.21" /> <!--  kg for small/big battery pack -->
-        <!-- servicebot's inertia tensor is approximated by a cylinder with homogeneous mass distribution
-             More details: http://en.wikipedia.org/wiki/List_of_moment_of_inertia_tensors
-             m = 2.4 kg; h = 0.09 m; r = 0.175 m
-             ixx = 1/12 * m * (3 * r^2 + h^2)
-             iyy = 1/12 * m * (3 * r^2 + h^2)
-             izz = 1/2 * m * r^2
-          -->
-        <inertia ixx="0.00057724" ixy="0.0" ixz="0.0" iyy="0.00057724" iyz="0.0" izz="0.00000597" />
-      </inertial>
     </link>
     <!-- Motor baglantı plakası2 -->
@@ -261,17 +195,4 @@
         <origin xyz="0.015 -0.176 -0.086" rpy="1.5707 0 ${M_PI}" />
       </collision>
-      <inertial>
-        <!-- COM experimentally determined -->
-        <origin xyz="0.05375 -0.00689  -0.1" />
-        <mass value="0.21" /> <!--  kg for small/big battery pack -->
-        <!-- servicebot's inertia tensor is approximated by a cylinder with homogeneous mass distribution
-             More details: http://en.wikipedia.org/wiki/List_of_moment_of_inertia_tensors
-             m = 2.4 kg; h = 0.09 m; r = 0.175 m
-             ixx = 1/12 * m * (3 * r^2 + h^2)
-             iyy = 1/12 * m * (3 * r^2 + h^2)
-             izz = 1/2 * m * r^2
-          -->
-        <inertia ixx="0.00057724" ixy="0.0" ixz="0.0" iyy="0.00057724" iyz="0.0" izz="0.00000597" />
-      </inertial>
     </link>
     <!-- Motor1 -->
@@ -297,17 +218,4 @@
         <origin xyz="0.03 -0.05 0.03" rpy="0 ${M_PI_2} ${M_PI_2}" />
       </collision>
-      <inertial>
-        <!-- COM experimentally determined -->
-        <origin xyz="0.05375 -0.00689  -0.1" />
-        <mass value="0.21" /> <!--  kg for small/big battery pack -->
-        <!-- servicebot's inertia tensor is approximated by a cylinder with homogeneous mass distribution
-             More details: http://en.wikipedia.org/wiki/List_of_moment_of_inertia_tensors
-             m = 2.4 kg; h = 0.09 m; r = 0.175 m
-             ixx = 1/12 * m * (3 * r^2 + h^2)
-             iyy = 1/12 * m * (3 * r^2 + h^2)
-             izz = 1/2 * m * r^2
-          -->
-        <inertia ixx="0.00057724" ixy="0.0" ixz="0.0" iyy="0.00057724" iyz="0.0" izz="0.00000597" />
-      </inertial>
     </link>
     <!-- right_motor -->
@@ -334,17 +242,4 @@
         <origin xyz="0.03 0.05 -0.03" rpy="0 ${-M_PI_2} ${M_PI_2}" />
       </collision>
-      <inertial>
-        <!-- COM experimentally determined -->
-        <origin xyz="0.05375 -0.00689  -0.1" />
-        <mass value="0.21" /> <!--  kg for small/big battery pack -->
-        <!-- servicebot's inertia tensor is approximated by a cylinder with homogeneous mass distribution
-             More details: http://en.wikipedia.org/wiki/List_of_moment_of_inertia_tensors
-             m = 2.4 kg; h = 0.09 m; r = 0.175 m
-             ixx = 1/12 * m * (3 * r^2 + h^2)
-             iyy = 1/12 * m * (3 * r^2 + h^2)
-             izz = 1/2 * m * r^2
-          -->
-        <inertia ixx="0.00057724" ixy="0.0" ixz="0.0" iyy="0.00057724" iyz="0.0" izz="0.00000597" />
-      </inertial>
     </link>
     <!-- left_reduktor_mil -->
@@ -371,17 +266,4 @@
         <origin xyz="-0.007 0.013 0.007" rpy="0 ${M_PI_2} -${M_PI_2}" />
       </collision>
-      <inertial>
-        <!-- COM experimentally determined -->
-        <origin xyz="0.05375 -0.00689  -0.1" />
-        <mass value="0.21" /> <!--  kg for small/big battery pack -->
-        <!-- servicebot's inertia tensor is approximated by a cylinder with homogeneous mass distribution
-             More details: http://en.wikipedia.org/wiki/List_of_moment_of_inertia_tensors
-             m = 2.4 kg; h = 0.09 m; r = 0.175 m
-             ixx = 1/12 * m * (3 * r^2 + h^2)
-             iyy = 1/12 * m * (3 * r^2 + h^2)
-             izz = 1/2 * m * r^2
-          -->
-        <inertia ixx="0.00057724" ixy="0.0" ixz="0.0" iyy="0.00057724" iyz="0.0" izz="0.00000597" />
-      </inertial>
     </link>
     <!-- right_reduktor_mil -->
@@ -407,100 +289,15 @@
         <origin xyz="-0.007 -0.013 -0.007" rpy="0 ${-M_PI_2} -${M_PI_2}" />
       </collision>
-      <inertial>
-        <!-- COM experimentally determined -->
-        <origin xyz="0 0 0" />
-        <mass value="0.21" /> <!--  kg for small/big battery pack -->
-        <!-- servicebot's inertia tensor is approximated by a cylinder with homogeneous mass distribution
-             More details: http://en.wikipedia.org/wiki/List_of_moment_of_inertia_tensors
-             m = 2.4 kg; h = 0.09 m; r = 0.175 m
-             ixx = 1/12 * m * (3 * r^2 + h^2)
-             iyy = 1/12 * m * (3 * r^2 + h^2)
-             izz = 1/2 * m * r^2
-          -->
-        <inertia ixx="0.00057724" ixy="0.0" ixz="0.0" iyy="0.00057724" iyz="0.0" izz="0.00000597" />
-      </inertial>
     </link>
     <!-- left_drive_wheel -->
-    <joint name="left_wheel_joint" type="continuous">
+    <xacro:wheel name="left_wheel" parent="left_reduktor_mil" xyz="0.079 -0.155 ${0.0725 + 0.0099}" rpy="0 ${M_PI_2} ${M_PI_2}">
       <!-- prismatic -->
       <origin xyz="0. 0.04 0.0" rpy="0 0 0" />
-      <parent link="left_reduktor_mil" />
-      <child link="left_drive_wheel" />
-      <axis xyz="0 1 0" />
-      <!-- <limit lower="-0.15" upper="0.15" effort="100" velocity="0.01" /> -->
-      <limit effort="100" velocity="20" />
-    </joint>
-    <link name="left_drive_wheel">
-      <visual>
-        <geometry>
-          <mesh filename="package://service_description/meshes/servis/reduktorteker.STL" scale="0.001 0.001 0.001" />
-        </geometry>
-        <!-- <origin xyz="-0.155 -0.079 ${0.0725 + 0.01}" rpy="0 1.5779 0" /> -->
-        <origin xyz="0.079 -0.155 ${0.0725 + 0.0099}" rpy="0 ${M_PI_2} ${M_PI_2}" />
-      </visual>
-      <collision>
-        <geometry>
-          <!-- <cylinder length="0.142" radius="0.006" /> -->
-          <mesh filename="package://service_description/meshes/servis/reduktorteker.STL" scale="0.001 0.001 0.001" />
-        </geometry>
-        <!-- <origin xyz="-0.155 -0.079 ${0.0725 + 0.01}" rpy="0 1.57079 0" /> -->
-        <origin xyz="0.079 -0.155 ${0.0725 + 0.0099}" rpy="0 ${M_PI_2} ${M_PI_2}" />
-      </collision>
-      <inertial>
-        <!-- COM experimentally determined -->
-        <origin xyz="0.05375 -0.00689  -0.1" />
-        <mass value="0.21" /> <!--  kg for small/big battery pack -->
-        <!-- servicebot's inertia tensor is approximated by a cylinder with homogeneous mass distribution
-             More details: http://en.wikipedia.org/wiki/List_of_moment_of_inertia_tensors
-             m = 2.4 kg; h = 0.09 m; r = 0.175 m
-             ixx = 1/12 * m * (3 * r^2 + h^2)
-             iyy = 1/12 * m * (3 * r^2 + h^2)
-             izz = 1/2 * m * r^2
-          -->
-        <inertia ixx="0.00057724" ixy="0.0" ixz="0.0" iyy="0.00057724" iyz="0.0" izz="0.00000597" />
-      </inertial>
-    </link>
+    </xacro:wheel>
     <!-- right_drive_wheel -->
-    <joint name="right_wheel_joint" type="continuous">
-      <!-- <origin xyz="-0.04 0.0 0.0" rpy="0 0 0" /> -->
+    <xacro:wheel name="right_wheel" parent="right_reduktor_mil" xyz="0.079 -0.155 ${0.0725 + 0.0099}" rpy="0 ${M_PI_2} ${-M_PI_2}">
+      <!-- prismatic -->
       <origin xyz="0.0 -0.04 0.0" rpy="0 0 0" />
-      <parent link="right_reduktor_mil" />
-      <child link="right_drive_wheel" />
-      <!-- <axis xyz="1 0 0" /> -->
-      <axis xyz="0 1 0" />
-      <!-- <limit lower="-0.15" upper="0.15" effort="100" velocity="0.01" /> -->
-      <limit effort="100" velocity="20" />
-    </joint>
-    <link name="right_drive_wheel">
-      <visual>
-        <geometry>
-          <mesh filename="package://service_description/meshes/servis/reduktorteker.STL" scale="0.001 0.001 0.001" />
-        </geometry>
-        <!-- <origin xyz="0.155 -0.079 -${0.0725 + 0.01}" rpy="0 -1.57079 0" /> -->
-        <origin xyz="0.079 0.155 -${0.0725 + 0.0099}" rpy="0 ${-M_PI_2} ${M_PI_2}" />
-      </visual>
-      <collision>
-        <geometry>
-          <!-- <cylinder length="0.142" radius="0.006" /> -->
-          <mesh filename="package://service_description/meshes/servis/reduktorteker.STL" scale="0.001 0.001 0.001" />
-        </geometry>
-        <!-- <origin xyz="0.155 -0.079 -${0.0725 + 0.01}" rpy="0 -1.57079 0" /> -->
-        <origin xyz="0.079 0.155 -${0.0725 + 0.0099}" rpy="0 ${-M_PI_2} ${M_PI_2}" />
-      </collision>
-      <inertial>
-        <!-- COM experimentally determined -->
-        <origin xyz="0 0 0" />
-        <mass value="0.21" /> <!--  kg for small/big battery pack -->
-        <!-- servicebot's inertia tensor is approximated by a cylinder with homogeneous mass distribution
-             More details: http://en.wikipedia.org/wiki/List_of_moment_of_inertia_tensors
-             m = 2.4 kg; h = 0.09 m; r = 0.175 m
-             ixx = 1/12 * m * (3 * r^2 + h^2)
-             iyy = 1/12 * m * (3 * r^2 + h^2)
-             izz = 1/2 * m * r^2
-          -->
-        <inertia ixx="0.00057724" ixy="0.0" ixz="0.0" iyy="0.00057724" iyz="0.0" izz="0.00000597" />
-      </inertial>
-    </link>
-    <!-- 3D camera -->
+    </xacro:wheel>
     <!-- Chaster wheel chassis1 -->
     <joint name="chaster_wheel_chassis_joint1" type="revolute">
@@ -529,17 +326,4 @@
         <origin xyz="-0.03 -0.03 -0.035" rpy="${M_PI_2} 0 ${M_PI_2}" />
       </collision>
-      <inertial>
-        <!-- COM experimentally determined -->
-        <origin xyz="0.0 0.0 0.0" />
-        <mass value="0.21" /> <!--  kg for small/big battery pack -->
-        <!-- servicebot's inertia tensor is approximated by a cylinder with homogeneous mass distribution
-             More details: http://en.wikipedia.org/wiki/List_of_moment_of_inertia_tensors
-             m = 2.4 kg; h = 0.09 m; r = 0.175 m
-             ixx = 1/12 * m * (3 * r^2 + h^2)
-             iyy = 1/12 * m * (3 * r^2 + h^2)
-             izz = 1/2 * m * r^2
-          -->
-        <inertia ixx="0.00057724" ixy="0.0" ixz="0.0" iyy="0.00057724" iyz="0.0" izz="0.00000597" />
-      </inertial>
     </link>
     <!-- Chaster wheel chassis2 -->
@@ -569,17 +353,4 @@
         <origin xyz="-0.03 -0.03 -0.035" rpy="${M_PI_2} 0 ${M_PI_2}" />
       </collision>
-      <inertial>
-        <!-- COM experimentally determined -->
-        <origin xyz="0.0 0.0 0.0" />
-        <mass value="0.21" /> <!--  kg for small/big battery pack -->
-        <!-- servicebot's inertia tensor is approximated by a cylinder with homogeneous mass distribution
-             More details: http://en.wikipedia.org/wiki/List_of_moment_of_inertia_tensors
-             m = 2.4 kg; h = 0.09 m; r = 0.175 m
-             ixx = 1/12 * m * (3 * r^2 + h^2)
-             iyy = 1/12 * m * (3 * r^2 + h^2)
-             izz = 1/2 * m * r^2
-          -->
-        <inertia ixx="0.00057724" ixy="0.0" ixz="0.0" iyy="0.00057724" iyz="0.0" izz="0.00000597" />
-      </inertial>
     </link>
     <!-- Chaster wheel chassis3 -->
@@ -609,17 +380,4 @@
         <origin xyz="-0.03 -0.03 -0.035" rpy="${M_PI_2} 0 ${M_PI_2}" />
       </collision>
-      <inertial>
-        <!-- COM experimentally determined -->
-        <origin xyz="0.0 0.0 0.0" />
-        <mass value="0.20" /> <!--  kg for small/big battery pack -->
-        <!-- servicebot's inertia tensor is approximated by a cylinder with homogeneous mass distribution
-             More details: http://en.wikipedia.org/wiki/List_of_moment_of_inertia_tensors
-             m = 2.4 kg; h = 0.09 m; r = 0.175 m
-             ixx = 1/12 * m * (3 * r^2 + h^2)
-             iyy = 1/12 * m * (3 * r^2 + h^2)
-             izz = 1/2 * m * r^2
-          -->
-        <inertia ixx="0.00057724" ixy="0.0" ixz="0.0" iyy="0.00057724" iyz="0.0" izz="0.00000597" />
-      </inertial>
     </link>
     <!-- Chaster wheel1 -->
@@ -663,17 +421,4 @@
         <origin xyz="-0.31 0.32 -0.03" rpy="0 0 -${pi/2}" />
       </collision>
-      <inertial>
-        <!-- COM experimentally determined -->
-        <origin xyz="0.0 0.0 0.0" />
-        <mass value="30" /> <!--  kg for small/big battery pack -->
-        <!-- servicebot's inertia tensor is approximated by a cylinder with homogeneous mass distribution
-             More details: http://en.wikipedia.org/wiki/List_of_moment_of_inertia_tensors
-             m = 2.4 kg; h = 0.09 m; r = 0.175 m
-             ixx = 1/12 * m * (3 * r^2 + h^2)
-             iyy = 1/12 * m * (3 * r^2 + h^2)
-             izz = 1/2 * m * r^2
-          -->
-        <inertia ixx="0.0057724" ixy="0.0" ixz="0.0" iyy="0.0057724" iyz="0.0" izz="0.0000597" />
-      </inertial>
     </link>
     <!-- Rplidar-->
@@ -693,6 +438,4 @@
       <origin xyz=" 0.128 0.00  0.19" rpy="0 0 0" />
     </xacro:imu>
-    <!-- gazebo simulation plugin -->
-    <xacro:servicebot_sim />
   </xacro:macro>
 </robot>

File: src/service_description/urdf/xacro/wheel.xacro (robot description, xacro)
@@ -1,5 +1,5 @@
 <?xml version="1.0" encoding="UTF-8"?>
-<robot xmlns:xacro="http://www.ros.org/wiki/xacro" name="servicebot">
-    <xacro:macro name="wheel" params="name parent *origin">
+<robot xmlns:xacro="http://www.ros.org/wiki/xacro">
+    <xacro:macro name="wheel" params="name parent xyz rpy *origin">
         <joint name="${name}_joint" type="continuous">
             <xacro:insert_block name="origin" />
@@ -10,24 +10,18 @@
         <link name="${name}">
             <visual>
-                <origin xyz="0.08 -0.15 0.08" rpy="0 1.57 1.57" />
                 <geometry>
-                    <mesh filename="package://service_description_clean/meshes/servis/wheel.STL" scale="0.001 0.001 0.001" />
+                    <mesh filename="package://service_description/meshes/servis/reduktorteker.STL" scale="0.001 0.001 0.001" />
                 </geometry>
+                <!-- <origin xyz="-0.155 -0.079 ${0.0725 + 0.01}" rpy="0 1.5779 0" /> -->
+                <origin xyz="${xyz}" rpy="${rpy}" />
             </visual>
-        </link>
-    </xacro:macro>
-    <xacro:macro name="camera" params="name parent *origin">
-        <joint name="${name}_joint" type="fixed">
-            <xacro:insert_block name="origin" />
-            <parent link="${parent}" />
-            <child link="${name}" />
-        </joint>
-        <link name="${name}">
-            <visual>
-                <origin xyz="0.01 0 0" rpy="1.57 0 1.57" />
+            <collision>
                 <geometry>
-                    <mesh filename="package://service_description_clean/meshes/sensors/d435.dae" />
+                    <!-- <cylinder length="0.142" radius="0.006" /> -->
+                    <mesh filename="package://service_description/meshes/servis/reduktorteker.STL" scale="0.001 0.001 0.001" />
                 </geometry>
-            </visual>
+                <!-- <origin xyz="-0.155 -0.079 ${0.0725 + 0.01}" rpy="0 1.57079 0" /> -->
+                <origin xyz="0.079 -0.155 ${0.0725 + 0.0099}" rpy="0 ${M_PI_2} ${M_PI_2}" />
+            </collision>
         </link>
     </xacro:macro>
