Commit message: refactor: urdf and launch files edit

File: src/service_description/urdf/xacro/depth_camera.xacro (robot description, xacro)
@@ -2,5 +2,5 @@
 <robot xmlns:xacro="http://www.ros.org/wiki/xacro" name="servicebot">
 	<xacro:macro name="depth_camera" params="name parent *origin">
-		<xacro:property name="depth_camera_link" value="0.05" />
+		<xacro:property name="depth_camera" value="0.05" />
 		<joint name="${name}_joint" type="fixed">
 			<axis xyz="0 1 0" />
@@ -21,11 +21,11 @@
 		<link name="${name}_link">
 			<collision>
-				<origin xyz="0 0 0" rpy="0 0 0" />
+				<origin xyz="0 0.02 0" rpy="${M_PI_2} 0 ${M_PI_2}" />
 				<geometry>
-					<box size="${depth_camera_link} ${depth_camera_link} ${depth_camera_link}" />
+					<box size="${depth_camera} ${depth_camera} ${2*depth_camera}" />
 				</geometry>
 			</collision>
 			<visual>
-				<origin xyz="0 -0.0175 0" rpy="1.570796 0 1.570796" />
+				<origin xyz="0 0.02 0" rpy="${M_PI_2} 0 ${M_PI_2}" />
 				<geometry>
 					<mesh filename="package://service_description/meshes/sensors/d435.dae" />

File: src/service_description/urdf/xacro/servicebot.urdf.xacro (robot description, xacro)
@@ -296,5 +296,5 @@
     </xacro:wheel>
     <!-- right_drive_wheel -->
-    <xacro:wheel name="right_wheel" parent="right_reduktor_mil" xyz="0.079 -0.155 ${0.0725 + 0.0099}" rpy="0 ${M_PI_2} ${-M_PI_2}">
+    <xacro:wheel name="right_wheel" parent="right_reduktor_mil" xyz="0.079 0.155 -${0.0725 + 0.0099}" rpy="0 ${-M_PI_2} ${M_PI_2}">
       <!-- prismatic -->
       <origin xyz="0.0 -0.04 0.0" rpy="0 0 0" />
