Commit message: refactor :wheel xacro file edit

File: src/service_description/urdf/xacro/wheel.xacro (robot description, xacro)
@@ -22,5 +22,5 @@
                 </geometry>
                 <!-- <origin xyz="-0.155 -0.079 ${0.0725 + 0.01}" rpy="0 1.57079 0" /> -->
-                <origin xyz="0.079 -0.155 ${0.0725 + 0.0099}" rpy="0 ${M_PI_2} ${M_PI_2}" />
+                <origin xyz="${xyz}" rpy="${rpy}" />
             </collision>
         </link>
